File: 02-PROJECTS/00-electrical/cad/icu-carrier/icu-carrier.kicad_sch (KiCad schematic)
At the start: 98 parts, among them J1 DT13-06PA, J2 backlight out, J3 DT13-12PA, J4 BT817 EVE bridge header, J5 Teensy 4.1 socket - 2 x 24 fe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, Q1 SQD50P06 class, >= 60 V, Q2 MMBT3904, SW1 IC22, U1 LMR36015-Q1 class - 60 V in, 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, U2 VN5E class, >= 6 A - DNP, U3 TCAN1042HVDRQ1, U4 LM393, U5 74LVC1G17, U7 LSM6DSO / ICM-42688-P, U8 XIAO ESP32C3

Commit message: pbc part 1
Parts:
- removed U1: LMR36015-Q1 class - 60 V in, 1.5 A, symbol icu-carrier:BUCK_60V_5V
- added C20: 4.7u 100V X7R, Capacitor_SMD:C_1210_3225Metric, symbol icu-carrier:C
- added C21, C22: 220n 100V, Capacitor_SMD:C_0805_2012Metric, symbol icu-carrier:C
- added C23: 22u 10V X7R, Capacitor_SMD:C_1206_3216Metric, symbol icu-carrier:C
- added C24: 100n 16V, Capacitor_SMD:C_0805_2012Metric, symbol icu-carrier:C
- added C25: 1u 16V, Capacitor_SMD:C_0805_2012Metric, symbol icu-carrier:C
- added C26: 20p C0G, Capacitor_SMD:C_0805_2012Metric, symbol icu-carrier:C
- added L2: 2.2u XAL4020-222, Inductor_SMD:L_Coilcraft_XAL4020-XXX, symbol icu-carrier:L
- added R41: 100k 1%, Resistor_SMD:R_0805_2012Metric, symbol icu-carrier:R
- added R42: 24.9k 1%, Resistor_SMD:R_0805_2012Metric, symbol icu-carrier:R
- added R43: 100k, Resistor_SMD:R_0805_2012Metric, symbol icu-carrier:R
- added U1: LMR36015FSCQ-Q1, Package_DFN_QFN:Texas_RNX0012C_VQFN-14-11-1EP_2x3mm_P0.5mm_EP0.25x1.825mm, symbol icu-carrier:LMR36015
- C1: footprint (none) -> Capacitor_SMD:CP_Elec_8x10
- C10, C11, C12, C13, C14, C15, C16, C17, C18, C19, C3, C4, C5, C6, C7, C8, C9: footprint (none) -> Capacitor_SMD:C_0805_2012Metric
- C2: footprint (none) -> Capacitor_SMD:C_1206_3216Metric
- D1, D10, D2, D20, D21, D22, D3, D4, D5, D6, D7, D8, D9, Q2: footprint (none) -> Package_TO_SOT_SMD:SOT-23
- D23: renamed from D1; footprint (none) -> Diode_SMD:D_SMA
- D24: renamed from D2; footprint (none) -> Diode_SMD:D_SMB
- D25: renamed from D3; footprint (none) -> Diode_SMD:D_SMA
- D26: renamed from D4; footprint (none) -> Diode_SMD:D_SMB
- F1: footprint (none) -> Fuse:Fuse_1206_3216Metric
- J1: footprint (none) -> Connector_PinHeader_2.54mm:PinHeader_2x03_P2.54mm_Vertical
- J2, JP1, JP2, JP3: footprint (none) -> Connector_PinHeader_2.54mm:PinHeader_1x02_P2.54mm_Vertical
- J3: footprint (none) -> Connector_PinHeader_2.54mm:PinHeader_2x06_P2.54mm_Vertical
- J4: footprint (none) -> Connector_PinHeader_2.54mm:PinHeader_1x10_P2.54mm_Vertical
- J5: footprint (none) -> icu-carrier:Teensy41_Socket; Note functional pins only - no Teensy pin numbers are asserted -> real Teensy 4.1 pads - pin map D-377, icu_channels.teensy_p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
- JP8A1: renamed from JP8A; footprint (none) -> Connector_PinHeader_2.54mm:PinHeader_1x02_P2.54mm_Vertical
- JP8B1: renamed from JP8B; footprint (none) -> Connector_PinHeader_2.54mm:PinHeader_1x02_P2.54mm_Vertical
- L1: footprint (none) -> Inductor_SMD:L_CommonModeChoke_Coilank_ACM2012
- Q1: footprint (none) -> Package_TO_SOT_SMD:TO-252-2
- R1, R10, R12, R13, R14, R15, R16, R17, R18, R19, R2, R20, R21, R22, R23, R24, R25, R26, R27, R28, R3, R31, R32, R33, R34, R35, R36, R37, R38, R39, R4, R40, R5, R7, R8, R9: footprint (none) -> Resistor_SMD:R_0805_2012Metric
- R11, R6: footprint (none) -> Resistor_SMD:R_2512_6332Metric
- R29, R30: footprint (none) -> Resistor_SMD:R_1210_3225Metric
- SW1: footprint (none) -> Connector_JST:JST_XH_B2B-XH-A_1x02_P2.50mm_Vertical
- U3, U4: footprint (none) -> Package_SO:JEITA_SOIC-8_3.9x4.9mm_P1.27mm
- U5: footprint (none) -> Package_TO_SOT_SMD:SOT-23-5
- U7: footprint (none) -> Connector_PinHeader_2.54mm:PinHeader_1x06_P2.54mm_Vertical
- U8: footprint (none) -> RF_Module:MCU_Seeed_ESP32C3
Connections:
- net +12V_BL: no longer D25.2 (A), F1.1, J1.6 (Pin_6), Q1.3 (S), R1.1
- net +12V_LOGIC: now also C20.1, C21.1, C22.1, U1.10 (VIN), U1.2 (VIN), U1.9 (EN); no longer D23.2 (A), J1.1 (Pin_1)
- net +3V3: now also J5.15 (3V3), J5.46 (3V3), R43.1; no longer C1.2, C10.1, C10.2, C11.1, C11.2, C12.1, C12.2, C13.1, C13.2, C14.1, C14.2, C15.2, C16.2, C17.2, C18.2, C19.2, C2.2, C3.2, C4.2, C5.1, C5.2, C6.1, C6.2, C7.1, C7.2, C8.1, C8.2, C9.1, C9.2, D1.1 (A), D1.3 (COM), D10.1 (A), D10.3 (COM), D2.1 (A), D2.3 (COM), D20.1 (K), D21.1 (A), D22.1 (A), D24.1 (A1), D26.1 (A1), D3.1 (A), D3.3 (COM), D4.1 (A), D4.3 (COM), D5.1 (A), D5.3 (COM), D6.1 (A), D6.3 (COM), D7.1 (A), D7.3 (COM), D8.1 (A), D8.3 (COM), D9.1 (A), D9.3 (COM), J1.3 (Pin_3), J2.2 (Pin_2), J4.2 (GND), J5.1 (IC01_ADC), J5.10 (IC14_ADC), J5.2 (IC02_ADC), J5.3 (IC03_ADC), J5.4 (IC05_ADC), J5.5 (IC06_DIG), J5.6 (IC07_ADC), J5.7 (IC09_DIG), J5.8 (IC10_DIG), J5.9 (IC11_DIG), JP8A1.2, Q2.2 (E), R10.1, R10.2, R12.2, R13.1, R13.2, R14.2, R15.1, R15.2, R16.2, R17.1, R17.2, R19.2, R20.1, R20.2, R21.2, R22.1, R22.2, R23.2, R24.1, R24.2, R25.2, R26.1, R26.2, R27.2, R28.1, R28.2, R32.2, R35.1, R37.2, R4.2, R5.2, R7.2, R8.1, R8.2, R9.2, SW1.1, U3.2 (GND), U4.4 (V-), U4.5 (+), U4.6 (-), U5.3 (GND), U7.2 (GND), U8.2 (GND)
- net +5V: now also J5.48 (VIN), C23.1, C26.1, L2.2, R41.1
- net BL_EN: now also J5.28 (BL_EN); no longer J5.32 (BL_EN)
- net BT817_INT: now also J5.16 (BT817_INT); no longer J5.22 (BT817_INT)
- net BT817_PD: now also J5.11 (BT817_PD); no longer J5.23 (BT817_PD)
- net CAN_RXD: now also J5.45 (CAN_RXD); no longer J5.14 (CAN_RXD)
- net CAN_STB: now also J5.24 (CAN_STB); no longer J5.15 (CAN_STB)
- net CAN_TXD: now also J5.44 (CAN_TXD); no longer J5.13 (CAN_TXD)
- net I2C_SCL: now also J5.41 (I2C_SCL); no longer J5.24 (I2C_SCL)
- net I2C_SDA: now also J5.40 (I2C_SDA); no longer J5.25 (I2C_SDA)
- net IC04_CAP: now also J5.4 (IC04_CAP); no longer D20.2 (A), D21.3 (COM), J3.4 (Pin_4), J5.11 (IC04_CAP), R29.1, R29.2, R30.1, R30.2, R33.2, U4.3 (+)
- net IC08_CAP: now also J5.5 (IC08_CAP); no longer J5.12 (IC08_CAP)
- net ICU_B8: no longer JP8B1.2, R36.1
- net IMU_INT: now also J5.25 (IMU_INT); no longer J5.26 (IMU_INT)
- net PAGE_BTN: now also J5.17 (PAGE_BTN); no longer J5.31 (PAGE_BTN)
- net PG_5V: now also J5.29 (PG_5V), R43.2, U1.8 (PG); no longer J5.33 (PG_5V)
- net RADIO_BOOT: now also J5.27 (RADIO_BOOT); no longer J5.30 (RADIO_BOOT)
- net RADIO_EN: now also J5.26 (RADIO_EN); no longer J5.29 (RADIO_EN)
- net RADIO_RX: now also J5.10 (RADIO_RX); no longer J5.28 (RADIO_RX)
- net RADIO_TX: now also J5.9 (RADIO_TX); no longer J5.27 (RADIO_TX)
- net QSPI_CS renamed SPI_CS
- net SPI_CS: now also J5.12 (SPI_CS); no longer J5.16 (QSPI_CS)
- net QSPI_IO0 renamed BT_IO2
- net BT_IO2: now also J4.7 (QSPI_IO2); no longer J4.5 (QSPI_IO0)
- net QSPI_IO1 renamed BT_IO3
- net BT_IO3: now also J4.8 (QSPI_IO3); no longer J4.6 (QSPI_IO1)
- net QSPI_IO2 renamed IC06_DIG
- net IC06_DIG: now also C9.1, D5.3 (COM), R16.2, R17.1; no longer J4.7 (QSPI_IO2)
- net QSPI_IO3 renamed IC09_DIG
- net IC09_DIG: now also C11.1, D7.3 (COM), R21.2, R22.1; no longer J4.8 (QSPI_IO3)
- net QSPI_SCK renamed SPI_SCK
- net SPI_SCK: now also J5.35 (SPI_SCK); no longer J5.17 (QSPI_SCK)
- new net: D20.2 (A), D21.3 (COM), R30.1, R33.2, U4.3 (+)
- new net: R29.1, R30.2
- new net: JP8A1.2, R35.1
- new net: F1.1, Q1.3 (S), R1.1
- new net: D23.2 (A), J1.1 (Pin_1)
- new net: D25.2 (A), J1.6 (Pin_6)
- new net: JP8B1.2, R36.1
- new net BUCK_BOOT: C24.1, U1.4 (BOOT)
- new net BUCK_FB: C26.2, R41.2, R42.1, U1.7 (FB)
- new net BUCK_SW: C24.2, L2.1, U1.12 (SW), U1.3 (NC)
- new net BUCK_VCC: C25.1, U1.5 (VCC)
- new net GND: C1.2, C10.2, C11.2, C12.2, C13.2, C14.2, C15.2, C16.2, C17.2, C18.2, C19.2, C2.2, C20.2, C21.2, C22.2, C23.2, C25.2, C3.2, C4.2, C5.2, C6.2, C7.2, C8.2, C9.2, D1.1 (A), D10.1 (A), D2.1 (A), D20.1 (K), D21.1 (A), D22.1 (A), D24.1 (A1), D26.1 (A1), D3.1 (A), D4.1 (A), D5.1 (A), D6.1 (A), D7.1 (A), D8.1 (A), D9.1 (A), J1.3 (Pin_3), J2.2 (Pin_2), J4.2 (GND), J5.1 (GND), J5.34 (GND), J5.47 (GND), Q2.2 (E), R10.2, R13.2, R15.2, R17.2, R20.2, R22.2, R24.2, R26.2, R28.2, R32.2, R37.2, R4.2, R42.2, R5.2, R8.2, SW1.1, U1.1 (PGND), U1.11 (PGND), U1.6 (AGND), U3.2 (GND), U4.4 (V-), U4.5 (+), U4.6 (-), U5.3 (GND), U7.2 (GND), U8.2 (GND)
- new net IC01_ADC: C5.1, D1.3 (COM), J5.36 (IC01_ADC), R7.2, R8.1
- new net IC02_ADC: C6.1, D2.3 (COM), J5.37 (IC02_ADC), R10.1, R9.2
- new net IC03_ADC: C7.1, D3.3 (COM), J5.38 (IC03_ADC), R12.2, R13.1
- new net IC05_ADC: C8.1, D4.3 (COM), J5.39 (IC05_ADC), R14.2, R15.1
- new net IC07_ADC: C10.1, D6.3 (COM), J5.42 (IC07_ADC), R19.2, R20.1
- new net IC10_DIG: C12.1, D8.3 (COM), J5.22 (IC10_DIG), R23.2, R24.1
- new net IC11_DIG: C13.1, D9.3 (COM), J5.23 (IC11_DIG), R25.2, R26.1
- new net IC14_ADC: C14.1, D10.3 (COM), J5.43 (IC14_ADC), R27.2, R28.1
- new net ICU_B4: J3.4 (Pin_4), R29.2
- new net SPI_MISO: J4.6 (QSPI_IO1), J5.14 (SPI_MISO)
- new net SPI_MOSI: J4.5 (QSPI_IO0), J5.13 (SPI_MOSI)
Other:
- note added: "U1 (the 5 V buck) is drawn in full at the bottom of the sheet (F13)."
- note added: "U1 - the ICU's 5 V buck in full (work F13; record icu_channels IC12, parts P105 / P159). TI LMR36015-Q1 datasheet SNVSAY8D, typical application for 5 V: every value confirm until the part is chosen. Layout: input caps tight across both VIN/PGND pairs, SW copper short, CBOOT from BOOT to the SW-NC link, the feedback parts right at FB, AGND and PGND to the ground pour through vias."
