File: 02-PROJECTS/01-electrical/00-design/cad/dcu-carrier/dcu-carrier.kicad_pcb (KiCad board)
At the start: 2 copper layers, 180 x 80 mm, 136 parts, among them J1 DP-DCU DT13-06PA, J10 Teensy 4.1 socket - 2 x 24 fe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, J2 DP-DCU-C DT13-08PA, J3 cabin NTC lead, J4 panel ribbon 2x10 IDC, J5 blower pigtail, J6 servo header, J7 servo header, J8 servo header, J9 DP-DCU-B DT13-12PA, Q1 PMV37ENEA, Q2 PMV37ENEA, Q3 SQ2351ES class, >= 40 V confi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, Q4 MMBT3904, U1 LMR36015FSCQ-Q1, U10 BTT6200-4ESA, U11 DRV8962-Q1, U12 TCA9539-Q1, U2 TPS54560B-Q1, U3 TCAN1042HVDRQ1, U4 INA180A1, U5 BTS3011TE, U6 BTS3011TE, U7 BTS3011TE, U8 BTS3011TE, U9 BTT6050-1ERA

Commit message: Electrical: the DCU carrier's provisions for the open blocks' worst case - a second expander, the A/C clutch stage and pressure ADC, the radar alert input, the third comfort ground, all DNP (Y11)
Sheet rev 0.03: U13 TCA9539-Q1 at 0x75 on U12's bus (STATUS wired-OR on P00, radar alert on P01); U12 P17 drives U14 BTT6050-1ERA from V12C_RAW to DP-DCU-B 12; U15 ADS1115-Q1 with a TPS7B4250-Q1 sensor supply and PLACEHOLDER leads J11 / J12; DP-DCU-C 8 on PGND. Board rev 0.03 on the same outline: DRC 0/0/0, parity clean, ERC 0/0, check.py 0 mismatches. Rows SN16 / SN17 / SN25 / SN27, SN28-SN30 new, P149, P185-P187, F29's clause; the enclosure rebuilt from the new board (0 interferences, J12 grommet). Row Y11.

Co-Authored-By: Claude Fable 5.1 <noreply@anthropic.com>
Parts:
- added C38: 100n U13 VCC, Capacitor_SMD:C_0805_2012Metric, F.Cu at (154.9, 41.0)
- added C39: 100n U15 VDD, Capacitor_SMD:C_0805_2012Metric, F.Cu at (154.5, 13.9)
- added C40: 1u 50V, Capacitor_SMD:C_0805_2012Metric, F.Cu at (169.7, 37.6)
- added C41: 100n, Capacitor_SMD:C_0805_2012Metric, F.Cu at (165.2, 41.3)
- added C42: 2.2u, Capacitor_SMD:C_0805_2012Metric, F.Cu at (167.7, 41.3)
- added C43: 100n, Capacitor_SMD:C_0805_2012Metric, F.Cu at (158.2, 17.3)
- added C44: 100n, Capacitor_SMD:C_0805_2012Metric, F.Cu at (175.8, 13.9)
- added C45: 100n, Capacitor_SMD:C_0805_2012Metric, F.Cu at (176.0, 10.0)
- added D10: BAT54S, Package_TO_SOT_SMD:SOT-23, F.Cu at (168.0, 13.9)
- added D11: BAT54S, Package_TO_SOT_SMD:SOT-23, F.Cu at (166.0, 10.0)
- added D9: BAT54S, Package_TO_SOT_SMD:SOT-23, F.Cu at (158.2, 13.9)
- added J11: A/C pressure transducer lead - PLACEHOLDER, Connector_JST:JST_XH_B3B-XH-A_1x03_P2.50mm_Vertical, F.Cu at (173.9, 38.0)
- added J12: radar alert lead - PLACEHOLDER, Connector_JST:JST_XH_B2B-XH-A_1x02_P2.50mm_Vertical, F.Cu at (166.5, 3.40)
- added R59: 4.7k, Resistor_SMD:R_0805_2012Metric, B.Cu at (67.4, 30.7)
- added R60: 10k off at reset, Resistor_SMD:R_0805_2012Metric, B.Cu at (67.4, 33.0)
- added R61: 4.7k DEN low, Resistor_SMD:R_0805_2012Metric, B.Cu at (69.6, 77.9)
- added R62: 1.2k IS unread, Resistor_SMD:R_0805_2012Metric, B.Cu at (67.4, 77.9)
- added R63: 47R PROFET ground, Resistor_SMD:R_0805_2012Metric, B.Cu at (71.8, 77.9)
- added R64: 10k, Resistor_SMD:R_0805_2012Metric, F.Cu at (161.4, 13.9)
- added R65: 20k, Resistor_SMD:R_0805_2012Metric, F.Cu at (163.7, 13.9)
- added R66: 10k, Resistor_SMD:R_0805_2012Metric, F.Cu at (171.2, 13.9)
- added R67: 20k, Resistor_SMD:R_0805_2012Metric, F.Cu at (173.5, 13.9)
- added R68: 10k, Resistor_SMD:R_0805_2012Metric, F.Cu at (169.2, 10.0)
- added R69: 47k, Resistor_SMD:R_0805_2012Metric, F.Cu at (171.5, 10.0)
- added R70: 22k, Resistor_SMD:R_0805_2012Metric, F.Cu at (173.7, 10.0)
- added U13: TCA9539-Q1, Package_SO:TSSOP-24_4.4x7.8mm_P0.65mm, F.Cu at (160.0, 41.0)
- added U14: BTT6050-1ERA, dcu-carrier:Infineon_PG-TSDSO-14-22, B.Cu at (62.5, 74.6)
- added U15: ADS1115-Q1, Package_SO:MSOP-10_3x3mm_P0.5mm, F.Cu at (150.0, 15.5)
- added U16: TPS7B4250-Q1, Package_TO_SOT_SMD:SOT-23-5, F.Cu at (166.3, 37.6)
Connections:
- J2 pad 8: unconnected-(J2-Pin_8-Pad8) -> PGND
- J9 pad 12: unconnected-(J9-Pin_12-Pad12) -> /AC_CLUTCH
- U12 pad 20: /SEAT_STATUS -> /AC_CLUTCH_CMD
Routing:
- net /I2C_SCL: track 72.4 -> 341.0 mm, vias 3 -> 8
- net /EXP_RESET: track 106.4 -> 323.0 mm, vias 4 -> 7
- net /I2C_SDA: track 77.1 -> 263.3 mm, vias 2 -> 18
- net /AC_IN: track 0.00 -> 98.3 mm, vias 0 -> 8
- net /EXP_INT: track 91.9 -> 186.8 mm, vias 2 -> 12
- net +3V3: track 384.1 -> 457.1 mm, vias 18 -> 26
- net /AC_CLUTCH_CMD: track 0.00 -> 68.8 mm, vias 0 -> 1
- net /RADAR_ALERT: track 0.00 -> 57.3 mm, vias 0 -> 2
- net +5V: track 234.7 -> 291.0 mm, vias 5 -> 11
- net +12V_LOGIC: track 264.7 -> 309.9 mm, vias 10 -> 15
- net /SENS_5V: track 0.00 -> 35.8 mm, vias 0 -> 2
- net /SENS_5V_ADC: track 0.00 -> 27.0 mm, vias 0 -> 2
- net /AC_PRESS_IN: track 0.00 -> 26.7 mm, vias 0 -> 1
- net /AC_PRESS_ADC: track 0.00 -> 20.2 mm
- net /AC_CLUTCH: track 0.00 -> 14.3 mm
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Other:
- board text added: "DCU carrier H-002 rev 0.03 (Y11) PROVISIONAL OUTLINE 180 x 80 - confirm at V-102 (D-455)"
- board text removed: "DCU carrier H-002 rev 0.02 (Y5)\nPROVISIONAL OUTLINE 180 x 80 - confirm at V-102 (D-455)"

Commit message: Electrical: the DCU carrier board re-laid for the 2 x 13 ribbon header - board rev 0.04 matches the sheet, DRC and parity zero (Y12)
J4 is the 26-way header of D-458, three pitches left of the old 2 x 10 so pins 7-26 sit on its pads; H1 moved to (4, 15); F1, R71, R72 and TP1 placed; R39 / R41 10 k (D-465). The seventeen header signals re-routed, GND one connected pour. Enclosure rebuilt with RIBBON_WAYS 26, 0 interferences. The attempt's scripts and its state note are kept in relay-attempt/y12 for this commit and removed with the row.

Co-Authored-By: Claude Opus 5.5 <noreply@anthropic.com>
Parts:
- added F1: PTC 0.5A hold 1206 - confirm, Fuse:Fuse_1206_3216Metric, F.Cu at (43.8, 3.60)
- added R71: 100R, Resistor_SMD:R_0805_2012Metric, F.Cu at (44.9, 11.8)
- added R72: 100R, Resistor_SMD:R_0805_2012Metric, F.Cu at (44.9, 7.30)
- added TP1: ribbon spare, TestPoint:TestPoint_Pad_D1.0mm, B.Cu at (39.0, 7.60)
- J4: value panel ribbon 2x10 IDC -> panel ribbon 2x13 IDC, keyed; footprint Connector_IDC:IDC-Header_2x10_P2.54mm_Vertical -> Connector_IDC:IDC-Header_2x13_P2.54mm_Vertical
- R39, R41: value 100k -> 10k
- moved R51 14.2 mm to (19.4, 13.7)
- moved H1 11.0 mm to (4.00, 15.0)
- moved C24 10.3 mm to (2.52, 24.5), turned to -90 degrees
- moved J4 7.62 mm to (6.38, 7.60)
- moved R3 3.39 mm to (5.25, 20.4)
- moved R54 3.31 mm to (8.55, 18.7)
- moved R53 1.97 mm to (2.50, 20.4)
- moved R52 0.56 mm to (8.55, 14.2)
Routing:
- net /I2C_SCL: track 341.0 -> 400.5 mm, vias 8 -> 9
- net /ENC_FAN_B: track 88.5 -> 115.2 mm
- net /PNL_SDA: track 0.00 -> 16.8 mm
- net /I2C_SDA: track 263.3 -> 249.9 mm
- net /COL3: track 101.3 -> 112.0 mm, vias 3 -> 2
- net /PNL_SCL: track 0.00 -> 10.6 mm
- net /ENC_TEMP_A: track 133.7 -> 143.9 mm
- net /ENC_FAN_A: track 74.7 -> 84.6 mm
- net /ROW1: track 89.0 -> 98.9 mm, vias 0 -> 1
- net /ROW3: track 89.7 -> 99.2 mm, vias 0 -> 1
- net /ROW2: track 121.5 -> 130.8 mm, vias 6 -> 7
- net /JOY_Y: track 30.9 -> 40.2 mm
- net /JOY_X: track 35.0 -> 43.9 mm, vias 0 -> 1
- net /ENC_TEMP_B: track 79.2 -> 88.2 mm, vias 0 -> 1
- net /ENC_SEAT_DRV_A: track 77.3 -> 85.7 mm, vias 1 -> 0
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Other:
- board text added: "DCU carrier H-002 rev 0.04 (Y12) PROVISIONAL OUTLINE 180 x 80 - confirm at V-102 (D-455)"
- board text removed: "DCU carrier H-002 rev 0.03 (Y11) PROVISIONAL OUTLINE 180 x 80 - confirm at V-102 (D-455)"

Commit message: Electrical: the panel board redrawn to the ruled control set and the DCU sheet renamed to the ribbon; both packaged for the bench order with the upper board (Y20)
panel rev 0.04: 180 x 84.76 mm with the controls where the sketch puts them, a 4 x 3 matrix, one centre encoder with push, two seat encoders, DPDT sprung window switches, the screen header behind its window with a supply jumper, the LED driver with 24 LEDs, the 26-way ribbon and the 2 x 6 plate header; ERC 0, DRC and parity 0, check.py 79 checks 0 mismatches. The DCU carrier's ribbon nets renamed (sheet, symbol pins, board net names only; DRC and parity 0, check.py 163 / 0); check.py's panel and dcu entries follow the record. Found and recorded: the window switches must be double-pole, the screen a 3.3 V-bus module, the seat symbol cannot sit in the knob's centre without a hollow-shaft encoder. Gerbers, drills and BOMs for the panel and upper boards under fab/ for Y18; the climate-unit mock-up's ribbon header at the drawn 16.5 mm, rebuilt clear.

Co-Authored-By: Claude Fable 5.1 <noreply@anthropic.com>
Connections:
- net /ENC_FAN_A renamed /ENC_CENTRE_A
- net /ENC_FAN_B renamed /ENC_CENTRE_B
- net /ENC_TEMP_A renamed /ENC_CENTRE_PUSH
- net /ENC_TEMP_B renamed /ROW4
