File: 02-PROJECTS/01-electrical/00-design/cad/dcu-carrier/dcu-carrier.kicad_sch (KiCad schematic)
At the start: 125 parts, among them J1 DP-DCU DT13-06PA, J10 Teensy 4.1 socket - 2 x 24 fe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, J2 DP-DCU-C DT13-08PA, J3 cabin NTC lead, J4 panel ribbon 2x10 IDC, J5 blower pigtail, J6 servo header, J7 servo header, J8 servo header, J9 DP-DCU-B DT13-12PA, Q1 PMV37ENEA, Q2 PMV37ENEA, Q3 SQ2351ES class, >= 40 V confi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, Q4 MMBT3904, U1 LMR36015FSCQ-Q1, U10 BTT6200-4ESA, U11 DRV8962-Q1, U12 TCA9539-Q1, U2 TPS54560B-Q1, U3 TCAN1042HVDRQ1, U4 INA180A1, U5 BTS3011TE, U6 BTS3011TE, U7 BTS3011TE, U8 BTS3011TE, U9 BTT6050-1ERA

Commit message: Electrical: the DCU carrier's provisional board - real packages, placed, routed, poured, DRC clean, STEP built (Y5); Y11 opened for the open blocks' worst case
180 x 80 mm provisional (confirm until V-102, CK26); BTS3011TE / BTT6050 / BTT6200 / DRV8962 / TPS54560B / INA180 / TCA9539 on their real pins; DT13 and PG-TSDSO footprints; COMFORT and PGND pours at 4 mm / 0.5 mm; DRC 0/0/0, ERC 0/0, check.py 0 mismatches. SN16 / SN17 / SN22 carry the stage facts; P177 / P178; CK26. Y11: a second expander so P17 serves 02.15 (b), the radar input, J2 pin 8 as 01.26's ground.

Co-Authored-By: Claude Fable 5.1 <noreply@anthropic.com>
Parts:
- added C35: 100n at pin 25 (VCC), Capacitor_SMD:C_0805_2012Metric, symbol dcu-carrier:C
- added C36: 10n 100V VM-PGND1 (TI 6-1), Capacitor_SMD:C_0805_2012Metric, symbol dcu-carrier:C
- added C37: 10n 100V VM-PGND3 (TI 6-1), Capacitor_SMD:C_0805_2012Metric, symbol dcu-carrier:C
- added R55, R56, R57: 1.5k confirm vs stall (W-332), Resistor_SMD:R_0805_2012Metric, symbol dcu-carrier:R
- added R58: 10k STATUS pull-up (BTS3011TE p.40), Resistor_SMD:R_0805_2012Metric, symbol dcu-carrier:R
- J1: footprint (none) -> dcu-carrier:DT13-06PA
- J2: footprint (none) -> dcu-carrier:DT13-08PA
- J3, J5: footprint (none) -> Connector_JST:JST_XH_B2B-XH-A_1x02_P2.50mm_Vertical
- J6, J7, J8: footprint (none) -> Connector_PinHeader_2.54mm:PinHeader_1x03_P2.54mm_Vertical
- J9: footprint (none) -> dcu-carrier:DT13-12PA
- L2: footprint (none) -> Inductor_SMD:L_Coilcraft_XAL7030-682
- U1: footprint (none) -> Package_DFN_QFN:Texas_RNX0012C_VQFN-14-11-1EP_2x3mm_P0.5mm_EP0.25x1.825mm
- U10: footprint (none) -> dcu-carrier:Infineon_PG-TSDSO-24-21
- U11: footprint (none) -> Package_SO:HTSSOP-44-1EP_6.1x14mm_P0.635mm_EP5.2x14mm_Mask4.31x8.26mm
- U2: footprint (none) -> Package_SO:HSOP-8-1EP_3.9x4.9mm_P1.27mm_EP2.41x3.1mm
- U5, U6, U7, U8: footprint Package_TO_SOT_SMD:TO-252-5_TabPin3 -> Package_TO_SOT_SMD:TO-252-5_TabPin6
- U9: footprint (none) -> dcu-carrier:Infineon_PG-TSDSO-14-22
Connections:
- net +12V_CMF: now also U9.TAB (VS); no longer U9.1 (VS)
- net +12V_LOGIC: now also U10.TAB (VS), U11.11 (VM), U11.12 (VM), U11.2 (VM), U11.21 (VM), C36.1, C37.1; no longer U10.1 (VS), U11.1 (VM)
- net +3V3: now also U11.33 (VREF), R58.1; no longer U11.8 (VREF)
- net GND: now also U11.13 (PGND4), U11.20 (PGND3), U11.22 (GND), U11.23 (GND), U11.27 (OCPM), U11.28 (MODE), U11.3 (PGND1), U11.38 (IN4), U11.45 (PAD), C35.2, C36.2, C37.2, R55.2, R56.2, R57.2; no longer U11.11 (PGND), U11.18 (IN4)
- net MH_DEN_R: now also U9.5 (DEN); no longer U9.3 (DEN)
- net MH_GND: now also U9.3 (GND); no longer U9.5 (GND)
- net MH_IN: now also U9.4 (IN); no longer U9.2 (IN)
- net MH_IS: now also U9.6 (IS); no longer U9.4 (IS)
- net MIRROR_HEAT: now also U9.10 (OUT), U9.11 (OUT), U9.12 (OUT); no longer U9.6 (OUT)
- net MIR_CLUTCH: now also U11.14 (OUT4), U11.15 (OUT4), U11.16 (OUT4); no longer U11.23 (OUT4)
- net MIR_COM: now also U11.4 (OUT1), U11.5 (OUT1), U11.6 (OUT1); no longer U11.20 (OUT1)
- net MIR_CPH: now also U11.44 (CPH); no longer U11.3 (CPH)
- net MIR_CPL: now also U11.43 (CPL); no longer U11.4 (CPL)
- net MIR_DVDD: now also U11.24 (DVDD), U11.25 (VCC), C35.1; no longer U11.5 (DVDD)
- net MIR_EN1: now also U11.37 (EN1); no longer U11.13 (EN1)
- net MIR_EN2: now also U11.36 (EN2); no longer U11.15 (EN2)
- net MIR_EN3: now also U11.35 (EN3); no longer U11.17 (EN3)
- net MIR_EN4: now also U11.34 (EN4); no longer U11.19 (EN4)
- net MIR_IN1: now also U11.41 (IN1); no longer U11.12 (IN1)
- net MIR_IN2: now also U11.40 (IN2); no longer U11.14 (IN2)
- net MIR_IN3: now also U11.39 (IN3); no longer U11.16 (IN3)
- net MIR_L: now also U11.7 (OUT2), U11.8 (OUT2), U11.9 (OUT2); no longer U11.21 (OUT2)
- net MIR_R: now also U11.17 (OUT3), U11.18 (OUT3), U11.19 (OUT3); no longer U11.22 (OUT3)
- net MIR_VCP: now also U11.1 (VCP); no longer U11.2 (VCP)
- net MIR_nFAULT: now also U11.26 (nFAULT); no longer U11.7 (nFAULT)
- net MIR_nSLEEP: now also U11.42 (nSLEEP); no longer U11.6 (nSLEEP)
- net SC_DRV_RTN: now also U7.6 (OUT)
- net SC_PASS_RTN: now also U8.6 (OUT)
- net SH_DRV_RTN: now also U5.6 (OUT)
- net SH_PASS_RTN: now also U6.6 (OUT)
- net WIN_DRV_DN: now also U10.20 (OUT1); no longer U10.12 (OUT1)
- net WIN_DRV_UP: now also U10.24 (OUT0); no longer U10.11 (OUT0)
- net WIN_DSEL0_R: now also U10.8 (DSEL0); no longer U10.7 (DSEL0)
- net WIN_DSEL1_R: now also U10.11 (DSEL1); no longer U10.8 (DSEL1)
- net WIN_GND: now also U10.4 (GND); no longer U10.10 (GND)
- net WIN_IN1_R: now also U10.5 (IN1); no longer U10.3 (IN1)
- net WIN_IN2_R: now also U10.9 (IN2); no longer U10.4 (IN2)
- net WIN_IN3_R: now also U10.10 (IN3); no longer U10.5 (IN3)
- net WIN_IS: now also U10.7 (IS); no longer U10.9 (IS)
- net WIN_PASS_DN: now also U10.13 (OUT3); no longer U10.14 (OUT3)
- net WIN_PASS_UP: now also U10.17 (OUT2); no longer U10.13 (OUT2)
- net SEAT_STATUS: now reaches U12.20 (P17)
- net SEAT_STATUS: now also U5.4 (STATUS), U6.4 (STATUS), U7.4 (STATUS), U8.4 (STATUS), R58.2
- net MIR_IPROPI renamed MIR_IPROPI1
- net MIR_IPROPI1: now also U11.32 (IPROPI1); no longer U11.9 (IPROPI)
- new net MIR_IPROPI2: R55.1, U11.31 (IPROPI2)
- new net MIR_IPROPI3: R56.1, U11.30 (IPROPI3)
- new net MIR_IPROPI4: R57.1, U11.29 (IPROPI4)
- no-connect marks 4 -> 3
Other:
- note added: "- BTS3011TE STATUS x4 wired-OR to P17 with one 10k pull-up: a latched thermal fault reads low; clearing it needs P17 driven high (3-7 mA per faulted part) with IN low - confirm the expander's drive."
- note added: "- DRV8962: charge-pump, DVDD and VCC bypass per TI table 6-1; RIPROPI 1.5k x4 puts ITRIP near 10 A (VREF 3.3 V, 212 uA/A) - confirm vs stall (W-332)."
- note added: "- Module pin numbers are now the datasheets' (cad/pin_tables.csv, check.py); every footprint is stock KiCad or drawn from the vendor drawing - confirm against the parts in hand (R11)."
- note added: "- The enclosure: V-102 is unmeasured, so the board outline is PROVISIONAL (170 x 80 mm, four M3; sized by the three DT13 flanges) - confirm."
- note added: "NO-CONNECTS: DP-DCU-B 12 and DP-DCU-C 8 are sealing plugs (cavities); TPS54560B EN floats high on its internal pull-up. Expander P17 now carries SEAT_STATUS (Y5)."
- note added: "SN16 seat heat driver - the four BTS3011TE STATUS pins (open-drain, latched thermal fault) are wired-OR on SEAT_STATUS to expander P17 through R58"
- note added: "SN17 mirror drive: DRV8962-Q1 on its 44 real pins - 3 half-bridges + channel 4 low FET as the clutch sink, IN4 tied low (D-360); MODE low = 140 ns edges, OCPM low = latch-off (an nSLEEP pulse clears it), VCC tied to DVDD; fed from logic 12 V"
- note removed: "- BTS3011TE pin 4 and any status pin: confirm against the Infineon datasheet; drawn as IN / VDD / DRAIN / SOURCE."
- note removed: "- DRV8962 charge-pump and DVDD values: confirm against TI datasheet section 9."
- note removed: "- Module pin NUMBERS except the Teensy pads: functional blocks, fixed against each datasheet at layout (H-002)."
- note removed: "- The enclosure: V-102 is unmeasured, so the board has no outline yet."
- note removed: "NO-CONNECTS: DP-DCU-B 12 and DP-DCU-C 8 are sealing plugs (cavities); expander P17 is spare; TPS54560B EN floats high on its internal pull-up."
- note removed: "SN16 seat heat driver"
- note removed: "SN17 mirror drive: 3 half-bridges + channel 4 low FET as the clutch sink, IN4 tied low (D-360); fed from logic 12 V"
- moved on the sheet: C31, C32, C33, D7, D8, J5, J6, J7, J8, J9, Q1, Q2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

Commit message: Electrical: the DCU carrier's provisions for the open blocks' worst case - a second expander, the A/C clutch stage and pressure ADC, the radar alert input, the third comfort ground, all DNP (Y11)
Sheet rev 0.03: U13 TCA9539-Q1 at 0x75 on U12's bus (STATUS wired-OR on P00, radar alert on P01); U12 P17 drives U14 BTT6050-1ERA from V12C_RAW to DP-DCU-B 12; U15 ADS1115-Q1 with a TPS7B4250-Q1 sensor supply and PLACEHOLDER leads J11 / J12; DP-DCU-C 8 on PGND. Board rev 0.03 on the same outline: DRC 0/0/0, parity clean, ERC 0/0, check.py 0 mismatches. Rows SN16 / SN17 / SN25 / SN27, SN28-SN30 new, P149, P185-P187, F29's clause; the enclosure rebuilt from the new board (0 interferences, J12 grommet). Row Y11.

Co-Authored-By: Claude Fable 5.1 <noreply@anthropic.com>
Parts:
- added C38: 100n U13 VCC, Capacitor_SMD:C_0805_2012Metric, symbol dcu-carrier:C
- added C39: 100n U15 VDD, Capacitor_SMD:C_0805_2012Metric, symbol dcu-carrier:C
- added C40: 1u 50V, Capacitor_SMD:C_0805_2012Metric, symbol dcu-carrier:C
- added C41, C43, C44, C45: 100n, Capacitor_SMD:C_0805_2012Metric, symbol dcu-carrier:C
- added C42: 2.2u, Capacitor_SMD:C_0805_2012Metric, symbol dcu-carrier:C
- added D10, D11, D9: BAT54S, Package_TO_SOT_SMD:SOT-23, symbol dcu-carrier:BAT54S
- added J11: A/C pressure transducer lead - PLACEHOLDER, Connector_JST:JST_XH_B3B-XH-A_1x03_P2.50mm_Vertical, symbol dcu-carrier:Conn_01x03
- added J12: radar alert lead - PLACEHOLDER, Connector_JST:JST_XH_B2B-XH-A_1x02_P2.50mm_Vertical, symbol dcu-carrier:Conn_01x02
- added R59: 4.7k, Resistor_SMD:R_0805_2012Metric, symbol dcu-carrier:R
- added R60: 10k off at reset, Resistor_SMD:R_0805_2012Metric, symbol dcu-carrier:R
- added R61: 4.7k DEN low, Resistor_SMD:R_0805_2012Metric, symbol dcu-carrier:R
- added R62: 1.2k IS unread, Resistor_SMD:R_0805_2012Metric, symbol dcu-carrier:R
- added R63: 47R PROFET ground, Resistor_SMD:R_0805_2012Metric, symbol dcu-carrier:R
- added R64, R66, R68: 10k, Resistor_SMD:R_0805_2012Metric, symbol dcu-carrier:R
- added R65, R67: 20k, Resistor_SMD:R_0805_2012Metric, symbol dcu-carrier:R
- added R69: 47k, Resistor_SMD:R_0805_2012Metric, symbol dcu-carrier:R
- added R70: 22k, Resistor_SMD:R_0805_2012Metric, symbol dcu-carrier:R
- added U13: TCA9539-Q1, Package_SO:TSSOP-24_4.4x7.8mm_P0.65mm, symbol dcu-carrier:TCA9539-Q1
- added U14: BTT6050-1ERA, dcu-carrier:Infineon_PG-TSDSO-14-22, symbol dcu-carrier:BTT6050-1ERA
- added U15: ADS1115-Q1, Package_SO:MSOP-10_3x3mm_P0.5mm, symbol dcu-carrier:ADS1115-Q1
- added U16: TPS7B4250-Q1, Package_TO_SOT_SMD:SOT-23-5, symbol dcu-carrier:TPS7B4250-Q1
Connections:
- net +12V_LOGIC: now also C40.1, R68.1, U16.3 (VIN)
- net +3V3: now also C38.1, C39.1, D10.2 (K), D11.2 (K), D9.2 (K), U13.21 (A0), U13.24 (VCC), U15.8 (VDD)
- net +5V: now also C41.1, U16.1 (ADJ/EN)
- net EXP_INT: now also U13.1 (INT)
- net EXP_RESET: now also U13.3 (RESET)
- net GND: now also C38.2, C39.2, C40.2, C41.2, C42.2, C43.2, C44.2, C45.2, D10.1 (A), D11.1 (A), D9.1 (A), J11.3 (Pin_3), J12.2 (Pin_2), R60.2, R61.2, R62.2, R63.2, R65.2, R67.2, R70.2, U13.12 (GND), U13.2 (A1), U15.1 (ADDR), U15.3 (GND), U15.5 (AIN1), U15.7 (AIN3), U16.2 (GND), U16.5 (GND)
- net I2C_SCL: now also U13.22 (SCL), U15.10 (SCL)
- net I2C_SDA: now also U13.23 (SDA), U15.9 (SDA)
- net PGND: now also J2.8 (Pin_8)
- net SEAT_STATUS: now also U13.4 (P00); no longer U12.20 (P17)
- net V12C_RAW: now also U14.TAB (VS)
- net AC_CLUTCH: now reaches J9.12 (Pin_12)
- net AC_CLUTCH: now also U14.10 (OUT), U14.11 (OUT), U14.12 (OUT)
- new net AC_CLUTCH_CMD: R59.1, R60.1, U12.20 (P17)
- new net AC_DEN_R: R61.1, U14.5 (DEN)
- new net AC_GND: R63.1, U14.3 (GND)
- new net AC_IN: R59.2, U14.4 (IN)
- new net AC_IS: R62.1, U14.6 (IS)
- new net AC_PRESS_ADC: C43.1, D9.3 (COM), R64.2, R65.1, U15.4 (AIN0)
- new net AC_PRESS_IN: J11.2 (Pin_2), R64.1
- new net RADAR_ALERT: C45.1, D11.3 (COM), R69.2, R70.1, U13.5 (P01)
- new net RADAR_IN: J12.1 (Pin_1), R68.2, R69.1
- new net SENS_5V: C42.1, J11.1 (Pin_1), R66.1, U16.4 (VOUT)
- new net SENS_5V_ADC: C44.1, D10.3 (COM), R66.2, R67.1, U15.6 (AIN2)
- no-connect marks 3 -> 16
Other:
- note added: "- BTS3011TE STATUS x4 wired-OR to U13 P00 with one 10k pull-up: a latched thermal fault reads low; clearing it needs P00 driven high (3-7 mA per faulted part) with IN low - confirm the expander's drive."
- note added: "- The enclosure: V-102 is unmeasured, so the board outline is PROVISIONAL (180 x 80 mm, four M3; sized by the three DT13 flanges) - confirm."
- note added: "- The two PROFET IS lines (U9, U10) are not read: all 42 Teensy edge pins are used. Diagnostics stay off (DEN low), and so on the clutch stage U14 (Y11)."
- note added: "A/C CLUTCH block 02.15 (b) - DNP: U12 P17 -> U14 BTT6050-1ERA high side, fed from V12C_RAW, out on DP-DCU-B 12"
- note added: "A/C PRESSURE block 02.15 (b) - DNP: J11 transducer lead (0.5-4.5 V ratiometric, confirm) -> 10k / 20k -> U15 ADS1115-Q1 at 0x48; its 5 V from U16, which tracks +5V"
- note added: "DP-DCU-C 8 (J2 pin 8) is wired to PGND: block 01.26 (a), the third comfort ground (about 10 A per pin). The record keeps the cavity a sealing plug until 01.26 answers -"
- note added: "Every part in this box but U13 and C38 is DNP; each carries its reason in its Note field. Nothing here touches +12V_CMF; U14 and the GND / PGND rule (CONVENTIONS 5) hold."
- note added: "Fed from the comfort input ahead of D3 (the B560C carries only the servo rail and mirror heat); the coil returns at the compressor body (engine ground),"
- note added: "J11 is a PLACEHOLDER: 02.15 (b) gives the transducer's three wires no drop cavity (DP-DCU 1-6 used, DP-DCU-B 12 taken by the clutch) - confirm the harness path."
- note added: "NO-CONNECTS: TPS54560B EN floats high on its internal pull-up; U13 P03-P17 and U15 ALERT/RDY are unused. DP-DCU-B 12 (AC_CLUTCH) and DP-DCU-C 8 (PGND) are wired for blocks 02.15 / 01.26 (Y11)."
- note added: "No Teensy ADC pin is free (all 42 edge pins used, D-452), so the reading goes over I2C. AIN0 pressure, AIN2 the sensor supply (ratio = AIN0 / AIN2); AIN1 and AIN3 grounded, spare."
- note added: "PROVISIONS (Y11) - the open blocks' worst case, drawn in so an answer is a fitting change, not a redesign (D-455)"
- note added: "RADAR ALERT luxury 03.12 / Z-002 - DNP: J12 the receiver's alert lead -> 47k / 22k, 100n, BAT54S -> U13 P01; R68 wets an open-collector output"
- note added: "SN16 seat heat driver - the four BTS3011TE STATUS pins (open-drain, latched thermal fault) are wired-OR on SEAT_STATUS to expander U13 P00 through R58 (Y11)"
- note added: "Same I2C bus as U12 (R51 / R52). INT wired-OR on EXP_INT (both open-drain, one pull-up R53, Teensy 12); RESET shared on EXP_RESET (R54 holds both in reset):"
- note added: "The receiver sits behind the dash on its own feed (N103, A16); its alert line is local, not on a drop. Output type unknown: active-high 12 V reads high through the divider;"
- note added: "U13 second expander TCA9539-Q1 at 0x75 (A0 high, A1 low) - FITTED: P00 SEAT_STATUS (moved from U12 P17), P01 the radar alert"
- note added: "an open-collector output needs R68 fitted and reads low when it alerts. 12 V -> 3.8 V clamped by D11; 8 V still reads high (VIH 2.31 V at 3.3 V). J12 is a PLACEHOLDER - confirm."
- note added: "never through the DCU. F29 is 7.5 A for servo + mirror heat today: with a ~4 A coil it needs 10 A - confirm (V-101). The coil carries its own diode (EAS 60 mJ)."
- note added: "one pin left on the Teensy for neither, and a reset must leave every output stage off on both expanders at once. P02-P17 unused: firmware sets them outputs, low."
- note added: "the copper is there either way, the contact and its 14 AWG wire are fitted with the answer. DP-DCU-B 12 carries AC_CLUTCH (02.15 (b)); it stays a plug until then."
- note removed: "- BTS3011TE STATUS x4 wired-OR to P17 with one 10k pull-up: a latched thermal fault reads low; clearing it needs P17 driven high (3-7 mA per faulted part) with IN low - confirm the expander's drive."
- note removed: "- The enclosure: V-102 is unmeasured, so the board outline is PROVISIONAL (170 x 80 mm, four M3; sized by the three DT13 flanges) - confirm."
- note removed: "- The two PROFET IS lines are not read: all 42 Teensy edge pins are used. Diagnostics stay off (DEN low)."
- note removed: "NO-CONNECTS: DP-DCU-B 12 and DP-DCU-C 8 are sealing plugs (cavities); TPS54560B EN floats high on its internal pull-up. Expander P17 now carries SEAT_STATUS (Y5)."
- note removed: "SN16 seat heat driver - the four BTS3011TE STATUS pins (open-drain, latched thermal fault) are wired-OR on SEAT_STATUS to expander P17 through R58"

Commit message: Electrical: the panel's lights and the 26-way ribbon, the panel as a board, the DCU's release pull-downs (D-458, D-459, D-465)
Panel rev 0.03: IS31FL3236A at 0x3C driving 9 key LEDs and 26 knob-arc LEDs, dimmed with the dash; J1 2 x 13; the faceplate windows table in its README; DRC 0/0/0, enclosure rebuilt. DCU sheet rev 0.04: J4 2 x 13, R71 / R72 series, F1 PTC on +5V_PNL, R39 / R41 10 k pull-downs; the board re-lay is Y12. panel_ribbon 21-26, P155 / P157 / P173-P175, P192 / P193, H-008, SN23; rows R-APPLY-01.14 / 01.15.

Co-Authored-By: Claude Fable 5.1 <noreply@anthropic.com>
Parts:
- added F1: PTC 0.5A hold 1206 - confirm, Fuse:Fuse_1206_3216Metric, symbol dcu-carrier:Polyfuse
- added R71, R72: 100R, Resistor_SMD:R_0805_2012Metric, symbol dcu-carrier:R
- added TP1: ribbon spare, TestPoint:TestPoint_Pad_D1.0mm, symbol dcu-carrier:TestPoint
- J4: value panel ribbon 2x10 IDC -> panel ribbon 2x13 IDC, keyed; footprint Connector_IDC:IDC-Header_2x10_P2.54mm_Vertical -> Connector_IDC:IDC-Header_2x13_P2.54mm_Vertical; symbol dcu-carrier:Conn_02x10 -> dcu-carrier:Conn_02x13; Note (none) -> D-458: 26-way, 2 x 13 shrouded box header, keyed; pin-out p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
- R39, R41: value 100k -> 10k; Note (none) -> D-465: gate pull-down, 10k gate to source: holds the releas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
Connections:
- net +5V: now also F1.1
- net GND: now also J4.21, J4.23
- net I2C_SCL: now also R72.1
- net I2C_SDA: now also R71.1
- new net +5V_PNL: F1.2, J4.26
- new net PNL_SCL: J4.24, R72.2
- new net PNL_SDA: J4.22, R71.2
- new net SPARE: J4.25, TP1.1
Other:
- note added: "+5V_PNL: the logic +5V through F1, a 0.5 A-hold PTC, so a short on the panel trips F1 and never browns out the Teensy (VIN on +5V). SPARE (25) ends on TP1."
- note added: "Each ribbon line leaves through 100 R (R71 SDA, R72 SCL): a shorted or zapped ribbon conductor cannot drag the expanders' bus or a Teensy pin beyond what the"
- note added: "PANEL RIBBON LINES (D-458) - the panel's lights on the I2C bus, J4 21-26"
- note added: "The LED driver on the panel (IS31FL3236A, 0x3C) shares the bus with U12 (0x74), U13 (0x75) and U15 (0x48): R51 / R52 pull it up to +3V3 here."
- note added: "resistor allows (the driver has 8 kV HBM on its pins, the Teensy its own clamps; no room for a BAT54S by J4 - confirm). Run this bus at 100 kHz (about 1 m of ribbon) - confirm."

Commit message: Electrical: the panel board redrawn to the ruled control set and the DCU sheet renamed to the ribbon; both packaged for the bench order with the upper board (Y20)
panel rev 0.04: 180 x 84.76 mm with the controls where the sketch puts them, a 4 x 3 matrix, one centre encoder with push, two seat encoders, DPDT sprung window switches, the screen header behind its window with a supply jumper, the LED driver with 24 LEDs, the 26-way ribbon and the 2 x 6 plate header; ERC 0, DRC and parity 0, check.py 79 checks 0 mismatches. The DCU carrier's ribbon nets renamed (sheet, symbol pins, board net names only; DRC and parity 0, check.py 163 / 0); check.py's panel and dcu entries follow the record. Found and recorded: the window switches must be double-pole, the screen a 3.3 V-bus module, the seat symbol cannot sit in the knob's centre without a hollow-shaft encoder. Gerbers, drills and BOMs for the panel and upper boards under fab/ for Y18; the climate-unit mock-up's ribbon header at the drawn 16.5 mm, rebuilt clear.

Co-Authored-By: Claude Fable 5.1 <noreply@anthropic.com>
Connections:
- net ENC_FAN_A renamed ENC_CENTRE_A
- net ENC_FAN_B renamed ENC_CENTRE_B
- net ENC_TEMP_A renamed ENC_CENTRE_PUSH
- net ENC_TEMP_B renamed ROW4
Changed lines of the file:
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@@
 	(label "COL2" (at 396.24 332.74 180) (effects (font (size 1.27 1.27)) (justify right bottom)))
 	(wire (pts (xy 398.78 335.28) (xy 396.24 335.28)) (stroke (width 0) (type default)))
-	(label "ENC_FAN_A" (at 396.24 335.28 180) (effects (font (size 1.27 1.27)) (justify right bottom)))
+	(label "ENC_CENTRE_A"(at 396.24 335.28 180) (effects (font (size 1.27 1.27)) (justify right bottom)))
 	(wire (pts (xy 398.78 337.82) (xy 396.24 337.82)) (stroke (width 0) (type default)))
-	(label "ENC_TEMP_A" (at 396.24 337.82 180) (effects (font (size 1.27 1.27)) (justify right bottom)))
+	(label "ENC_CENTRE_PUSH"(at 396.24 337.82 180) (effects (font (size 1.27 1.27)) (justify right bottom)))
 	(wire (pts (xy 398.78 340.36) (xy 396.24 340.36)) (stroke (width 0) (type default)))
 	(label "ENC_SEAT_DRV_A" (at 396.24 340.36 180) (effects (font (size 1.27 1.27)) (justify right bottom)))
@@
 	(label "COL3" (at 416.56 332.74 0) (effects (font (size 1.27 1.27)) (justify left bottom)))
 	(wire (pts (xy 414.02 335.28) (xy 416.56 335.28)) (stroke (width 0) (type default)))
-	(label "ENC_FAN_B" (at 416.56 335.28 0) (effects (font (size 1.27 1.27)) (justify left bottom)))
+	(label "ENC_CENTRE_B"(at 416.56 335.28 0) (effects (font (size 1.27 1.27)) (justify left bottom)))
 	(wire (pts (xy 414.02 337.82) (xy 416.56 337.82)) (stroke (width 0) (type default)))
-	(label "ENC_TEMP_B" (at 416.56 337.82 0) (effects (font (size 1.27 1.27)) (justify left bottom)))
+	(label "ROW4"(at 416.56 337.82 0) (effects (font (size 1.27 1.27)) (justify left bottom)))
 	(wire (pts (xy 414.02 340.36) (xy 416.56 340.36)) (stroke (width 0) (type default)))
 	(label "ENC_SEAT_DRV_B" (at 416.56 340.36 0) (effects (font (size 1.27 1.27)) (justify left bottom)))
@@
 	(global_label "GND" (shape passive) (at 655.32 81.28 0) (effects (font (size 1.27 1.27)) (justify left)))
 	(wire (pts (xy 652.78 83.82) (xy 655.32 83.82)) (stroke (width 0) (type default)))
-	(label "ENC_FAN_B" (at 655.32 83.82 0) (effects (font (size 1.27 1.27)) (justify left bottom)))
+	(label "ENC_CENTRE_B"(at 655.32 83.82 0) (effects (font (size 1.27 1.27)) (justify left bottom)))
 	(wire (pts (xy 652.78 86.36) (xy 655.32 86.36)) (stroke (width 0) (type default)))
-	(label "ENC_FAN_A" (at 655.32 86.36 0) (effects (font (size 1.27 1.27)) (justify left bottom)))
+	(label "ENC_CENTRE_A"(at 655.32 86.36 0) (effects (font (size 1.27 1.27)) (justify left bottom)))
 	(wire (pts (xy 652.78 88.9) (xy 655.32 88.9)) (stroke (width 0) (type default)))
 	(label "ENC_SEAT_PASS_B" (at 655.32 88.9 0) (effects (font (size 1.27 1.27)) (justify left bottom)))
@@
 	(label "ENC_SEAT_DRV_A" (at 655.32 96.52 0) (effects (font (size 1.27 1.27)) (justify left bottom)))
 	(wire (pts (xy 652.78 99.06) (xy 655.32 99.06)) (stroke (width 0) (type default)))
-	(label "ENC_TEMP_B" (at 655.32 99.06 0) (effects (font (size 1.27 1.27)) (justify left bottom)))
+	(label "ROW4"(at 655.32 99.06 0) (effects (font (size 1.27 1.27)) (justify left bottom)))
 	(wire (pts (xy 652.78 101.6) (xy 655.32 101.6)) (stroke (width 0) (type default)))
-	(label "ENC_TEMP_A" (at 655.32 101.6 0) (effects (font (size 1.27 1.27)) (justify left bottom)))
+	(label "ENC_CENTRE_PUSH"(at 655.32 101.6 0) (effects (font (size 1.27 1.27)) (justify left bottom)))
 	(wire (pts (xy 652.78 104.14) (xy 655.32 104.14)) (stroke (width 0) (type default)))
 	(label "COL3" (at 655.32 104.14 0) (effects (font (size 1.27 1.27)) (justify left bottom)))
