File: 02-PROJECTS/01-electrical/00-design/cad/panel/panel.kicad_sch (KiCad schematic)
At the start: 25 parts, among them J1 panel ribbon 2x10 IDC, J2 illumination in, SW1 key - defog, SW10 encoder - fan, SW11 encoder - temperature, SW12 encoder - driver seat, SW13 encoder - passenger seat, SW2 key - hatch release, SW3 key - fuel-door release, SW4 key - HVAC mode, SW5 key - recirculate, SW6 key - window DRV up, SW7 key - window DRV down, SW8 key - window PASS up, SW9 key - window PASS down, U1 thumbstick - not chosen (P156)

Commit message: Electrical: the control panel's provisional board - both key styles as alternates, the backlight provided for, DRC clean, STEP built (Y6)
200 x 70 mm provisional outline (confirm until V-113); PEC11R footprint from the daxxn model; the thumbstick a placeholder (P156); J2 the illumination input; freerouting 0 unrouted; ERC 0/0, check.py 0 mismatches. Parts P155 corrected to the no-push encoder, P173-P175 added. Rows Y6, V-113, H-008 gates.

Co-Authored-By: Claude Fable 5.1 <noreply@anthropic.com>
Parts:
- added LED1: backlight defog - confirm, LED_SMD:LED_1206_3216Metric, symbol panel:LED
- added LED2: backlight hatch release - confirm, LED_SMD:LED_1206_3216Metric, symbol panel:LED
- added LED3: backlight fuel-door release - confirm, LED_SMD:LED_1206_3216Metric, symbol panel:LED
- added LED4: backlight HVAC mode - confirm, LED_SMD:LED_1206_3216Metric, symbol panel:LED
- added LED5: backlight recirculate - confirm, LED_SMD:LED_1206_3216Metric, symbol panel:LED
- added LED6: backlight window DRV up - confirm, LED_SMD:LED_1206_3216Metric, symbol panel:LED
- added LED7: backlight window DRV down - confirm, LED_SMD:LED_1206_3216Metric, symbol panel:LED
- added LED8: backlight window PASS up - confirm, LED_SMD:LED_1206_3216Metric, symbol panel:LED
- added LED9: backlight window PASS down - confirm, LED_SMD:LED_1206_3216Metric, symbol panel:LED
- added R1, R2, R3: 1k - confirm, Resistor_SMD:R_0805_2012Metric, symbol panel:R
- added SWB1: key (b) - defog, Connector_JST:JST_XH_B4B-XH-A_1x04_P2.50mm_Vertical, symbol panel:SW_Push_LED
- added SWB2: key (b) - hatch release, Connector_JST:JST_XH_B4B-XH-A_1x04_P2.50mm_Vertical, symbol panel:SW_Push_LED
- added SWB3: key (b) - fuel-door release, Connector_JST:JST_XH_B4B-XH-A_1x04_P2.50mm_Vertical, symbol panel:SW_Push_LED
- added SWB4: key (b) - HVAC mode, Connector_JST:JST_XH_B4B-XH-A_1x04_P2.50mm_Vertical, symbol panel:SW_Push_LED
- added SWB5: key (b) - recirculate, Connector_JST:JST_XH_B4B-XH-A_1x04_P2.50mm_Vertical, symbol panel:SW_Push_LED
- added SWB6: key (b) - window DRV up, Connector_JST:JST_XH_B4B-XH-A_1x04_P2.50mm_Vertical, symbol panel:SW_Push_LED
- added SWB7: key (b) - window DRV down, Connector_JST:JST_XH_B4B-XH-A_1x04_P2.50mm_Vertical, symbol panel:SW_Push_LED
- added SWB8: key (b) - window PASS up, Connector_JST:JST_XH_B4B-XH-A_1x04_P2.50mm_Vertical, symbol panel:SW_Push_LED
- added SWB9: key (b) - window PASS down, Connector_JST:JST_XH_B4B-XH-A_1x04_P2.50mm_Vertical, symbol panel:SW_Push_LED
- J2: footprint (none) -> Connector_JST:JST_XH_B2B-XH-A_1x02_P2.50mm_Vertical; Confirm (none) -> confirm: illumination lead from L3-S1 8 (DV53, PV94) - pin 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
- SW1, SW2, SW3, SW4, SW5, SW6, SW7, SW8, SW9: footprint (none) -> Button_Switch_THT:SW_PUSH_6mm_H13mm; Confirm (none) -> 03.14 (a): low-travel board switch under a faceplate cap, 6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
- SW10, SW11, SW12, SW13: footprint (none) -> panel:RotaryEncoder_Bourns_Vertical_PEC11R-4xxxF-Sxxxx; Confirm (none) -> confirm: PEC11R-4220F class; footprint drawn from the daxxn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
- U1: footprint (none) -> panel:Thumbstick_P156_Placeholder_2x04_P2.54mm; Confirm (none) -> PLACEHOLDER - confirm: P156 not chosen (ALPS RKJXV class). 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
Connections:
- net COL1: now also SWB1.1 (SW_1), SWB4.1 (SW_1), SWB7.1 (SW_1)
- net COL2: now also SWB2.1 (SW_1), SWB5.1 (SW_1), SWB8.1 (SW_1)
- net COL3: now also SWB3.1 (SW_1), SWB6.1 (SW_1), SWB9.1 (SW_1)
- net K1_11: now also SWB1.2 (SW_2)
- net K2_12: now also SWB2.2 (SW_2)
- net K3_13: now also SWB3.2 (SW_2)
- net K4_21: now also SWB4.2 (SW_2)
- net K5_22: now also SWB5.2 (SW_2)
- net K6_23: now also SWB6.2 (SW_2)
- net K7_31: now also SWB7.2 (SW_2)
- net K8_32: now also SWB8.2 (SW_2)
- net K9_33: now also SWB9.2 (SW_2)
- net ILLUM_12V: now reaches J2.1 (Pin_1)
- net ILLUM_12V: now also R1.1, R2.1, R3.1, SWB1.3 (LED_A), SWB2.3 (LED_A), SWB3.3 (LED_A), SWB4.3 (LED_A), SWB5.3 (LED_A), SWB6.3 (LED_A), SWB7.3 (LED_A), SWB8.3 (LED_A), SWB9.3 (LED_A)
- net ILLUM_GND: now reaches J2.2 (Pin_2)
- net ILLUM_GND: now also LED3.1 (K), LED6.1 (K), LED9.1 (K), SWB1.4 (LED_K), SWB2.4 (LED_K), SWB3.4 (LED_K), SWB4.4 (LED_K), SWB5.4 (LED_K), SWB6.4 (LED_K), SWB7.4 (LED_K), SWB8.4 (LED_K), SWB9.4 (LED_K)
- new net BL1_1: LED1.2 (A), R1.2
- new net BL1_2: LED1.1 (K), LED2.2 (A)
- new net BL1_3: LED2.1 (K), LED3.2 (A)
- new net BL2_1: LED4.2 (A), R2.2
- new net BL2_2: LED4.1 (K), LED5.2 (A)
- new net BL2_3: LED5.1 (K), LED6.2 (A)
- new net BL3_1: LED7.2 (A), R3.2
- new net BL3_2: LED7.1 (K), LED8.2 (A)
- new net BL3_3: LED8.1 (K), LED9.2 (A)
- no-connect marks 2 -> 0
Other:
- note added: "- Both key styles are drawn (SWn fitted, SWBn DNP); encoder and stick parts are confirm until V-113 and LP20."
- note added: "- ILLUM_12V / ILLUM_GND feed only DNP parts: the backlight and the (b) rings wait on 03.14 and 01.14."
- note added: "BACKLIGHT FOR KEY STYLE (a) - DNP: three strings of three LEDs off the illumination input, one string per matrix row"
- note added: "Each SWBn sits in parallel with SWn on the same column and diode: fit SW1-SW9 (style a, recommended) or SWB1-SWB9 (style b), never both. Ring LED 3-4 across the illumination input; a 12 V ring with its own resistor - confirm."
- note added: "KEY STYLE (b) - ALTERNATES, DNP: a 12-16 mm round button with a light ring, wired to the board on a 4-way JST-XH (luxury 03.14 open)"
- note added: "LEDn sits beside key SWn under its cap. ~5 mA per string at 13.8 V with white LEDs (13.8 - 3 x 2.9 V) / 1k. Values, colour and whether the keys are backlit at all wait on 03.14 and 01.14 - confirm."
- note added: "illumination in - its own lead from L3-S1 8, dims with the dash (DV53, PV94): feeds the backlight below (DNP)"
- note removed: "- ILLUM_12V / ILLUM_GND land nowhere yet: the lamps depend on the key style (a block)."
- note removed: "- Key switch, encoder shaft and thumbstick parts are placeholders until the faceplate is drawn."
- note removed: "illumination - its own lead from L3-S1 8, dims with the dash (DV53); the lamps wait on the key style"

Commit message: Electrical: the panel's lights and the 26-way ribbon, the panel as a board, the DCU's release pull-downs (D-458, D-459, D-465)
Panel rev 0.03: IS31FL3236A at 0x3C driving 9 key LEDs and 26 knob-arc LEDs, dimmed with the dash; J1 2 x 13; the faceplate windows table in its README; DRC 0/0/0, enclosure rebuilt. DCU sheet rev 0.04: J4 2 x 13, R71 / R72 series, F1 PTC on +5V_PNL, R39 / R41 10 k pull-downs; the board re-lay is Y12. panel_ribbon 21-26, P155 / P157 / P173-P175, P192 / P193, H-008, SN23; rows R-APPLY-01.14 / 01.15.

Co-Authored-By: Claude Fable 5.1 <noreply@anthropic.com>
Parts:
- removed R3: 1k - confirm, Resistor_SMD:R_0805_2012Metric, symbol panel:R
- added C1: 10u 16V X7R - confirm, Capacitor_SMD:C_0805_2012Metric, symbol panel:C
- added C2: 1u, Capacitor_SMD:C_0603_1608Metric, symbol panel:C
- added C3: 100n, Capacitor_SMD:C_0603_1608Metric, symbol panel:C
- added LED10: fan level 1 - confirm, LED_SMD:LED_0603_1608Metric, symbol panel:LED
- added LED11: fan level 2 - confirm, LED_SMD:LED_0603_1608Metric, symbol panel:LED
- added LED12: fan level 3 - confirm, LED_SMD:LED_0603_1608Metric, symbol panel:LED
- added LED13: fan level 4 - confirm, LED_SMD:LED_0603_1608Metric, symbol panel:LED
- added LED14: fan level 5 - confirm, LED_SMD:LED_0603_1608Metric, symbol panel:LED
- added LED15: fan level 6 - confirm, LED_SMD:LED_0603_1608Metric, symbol panel:LED
- added LED16: fan level 7 - confirm, LED_SMD:LED_0603_1608Metric, symbol panel:LED
- added LED17: temperature level 1 - confirm, LED_SMD:LED_0603_1608Metric, symbol panel:LED
- added LED18: temperature level 2 - confirm, LED_SMD:LED_0603_1608Metric, symbol panel:LED
- added LED19: temperature level 3 - confirm, LED_SMD:LED_0603_1608Metric, symbol panel:LED
- added LED20: temperature level 4 - confirm, LED_SMD:LED_0603_1608Metric, symbol panel:LED
- added LED21: temperature level 5 - confirm, LED_SMD:LED_0603_1608Metric, symbol panel:LED
- added LED22: temperature level 6 - confirm, LED_SMD:LED_0603_1608Metric, symbol panel:LED
- added LED23: temperature level 7 - confirm, LED_SMD:LED_0603_1608Metric, symbol panel:LED
- added LED24: driver seat cool 3 - confirm, LED_SMD:LED_0603_1608Metric, symbol panel:LED
- added LED25: driver seat cool 2 - confirm, LED_SMD:LED_0603_1608Metric, symbol panel:LED
- added LED26: driver seat cool 1 - confirm, LED_SMD:LED_0603_1608Metric, symbol panel:LED
- added LED27: driver seat heat 1 - confirm, LED_SMD:LED_0603_1608Metric, symbol panel:LED
- added LED28: driver seat heat 2 - confirm, LED_SMD:LED_0603_1608Metric, symbol panel:LED
- added LED29: driver seat heat 3 - confirm, LED_SMD:LED_0603_1608Metric, symbol panel:LED
- added LED30: passenger seat cool 3 - confirm, LED_SMD:LED_0603_1608Metric, symbol panel:LED
- added LED31: passenger seat cool 2 - confirm, LED_SMD:LED_0603_1608Metric, symbol panel:LED
- added LED32: passenger seat cool 1 - confirm, LED_SMD:LED_0603_1608Metric, symbol panel:LED
- added LED33: passenger seat heat 1 - confirm, LED_SMD:LED_0603_1608Metric, symbol panel:LED
- added LED34: passenger seat heat 2 - confirm, LED_SMD:LED_0603_1608Metric, symbol panel:LED
- added LED35: passenger seat heat 3 - confirm, LED_SMD:LED_0603_1608Metric, symbol panel:LED
- added TP1: ribbon spare, TestPoint:TestPoint_Pad_D1.5mm, symbol panel:TestPoint
- added U2: IS31FL3236A-TQLS4, Package_QFP:TQFP-48-1EP_7x7mm_P0.5mm_EP4.11x4.11mm, symbol panel:IS31FL3236A
- J1: value panel ribbon 2x10 IDC -> panel ribbon 2x13 IDC, keyed; footprint Connector_IDC:IDC-Header_2x10_P2.54mm_Vertical -> Connector_IDC:IDC-Header_2x13_P2.54mm_Vertical; symbol panel:Conn_02x10 -> panel:Conn_02x13; Confirm (none) -> 2 x 13 shrouded box header, 2.54 mm, keyed: the IDC plug go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
- J2: Confirm confirm: illumination lead from L3-S1 8 (DV53, PV94) - pin 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 -> DNP: fitted only with the style-(b) keys SWB1-9 (03.14), fo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; now not fitted
- LED1: value backlight defog - confirm -> key light defog - confirm; Confirm beside SW1 under its cap; colour and current from 03.14 - c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 -> by key SW1, under a faceplate window (panel/README.md); col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; now fitted
- LED2: value backlight hatch release - confirm -> key light hatch release - confirm; Confirm beside SW2 under its cap; colour and current from 03.14 - c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 -> by key SW2, under a faceplate window (panel/README.md); col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; now fitted
- LED3: value backlight fuel-door release - confirm -> key light fuel-door release - confirm; Confirm beside SW3 under its cap; colour and current from 03.14 - c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 -> by key SW3, under a faceplate window (panel/README.md); col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; now fitted
- LED4: value backlight HVAC mode - confirm -> key light HVAC mode - confirm; Confirm beside SW4 under its cap; colour and current from 03.14 - c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 -> by key SW4, under a faceplate window (panel/README.md); col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; now fitted
- LED5: value backlight recirculate - confirm -> key light recirculate - confirm; Confirm beside SW5 under its cap; colour and current from 03.14 - c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 -> by key SW5, under a faceplate window (panel/README.md); col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; now fitted
- LED6: value backlight window DRV up - confirm -> key light window DRV up - confirm; Confirm beside SW6 under its cap; colour and current from 03.14 - c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 -> by key SW6, under a faceplate window (panel/README.md); col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; now fitted
- LED7: value backlight window DRV down - confirm -> key light window DRV down - confirm; Confirm beside SW7 under its cap; colour and current from 03.14 - c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 -> by key SW7, under a faceplate window (panel/README.md); col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; now fitted
- LED8: value backlight window PASS up - confirm -> key light window PASS up - confirm; Confirm beside SW8 under its cap; colour and current from 03.14 - c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 -> by key SW8, under a faceplate window (panel/README.md); col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; now fitted
- LED9: value backlight window PASS down - confirm -> key light window PASS down - confirm; Confirm beside SW9 under its cap; colour and current from 03.14 - c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 -> by key SW9, under a faceplate window (panel/README.md); col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; now fitted
- R1: value 1k - confirm -> 10k; footprint Resistor_SMD:R_0805_2012Metric -> Resistor_SMD:R_0603_1608Metric; Confirm backlight string 1 series resistor: value from the LED chos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 -> R_EXT: IMAX = 58.5 x 1.3 V / R (p.11) = 7.6 mA per channel;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; now fitted
- R2: value 1k - confirm -> 100k; footprint Resistor_SMD:R_0805_2012Metric -> Resistor_SMD:R_0603_1608Metric; Confirm backlight string 2 series resistor: value from the LED chos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 -> SDB pull-up: enabled whenever +5V_PNL is up; registers powe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; now fitted
Connections:
- net BL2_1 is gone; now on net +5V_PNL: LED4.2 (A), R2.2
- net BL3_1 is gone; now on net +5V_PNL: LED7.2 (A)
- net GND: now also J1.21, J1.23, R1.2, C1.2, C2.2, C3.2, U2.18 (GND), U2.19 (GND), U2.33 (GND), U2.4 (GND), U2.40 (AD), U2.42 (GND), U2.43 (GND), U2.49 (PAD)
- net ILLUM_12V: no longer R1.1, R2.1
- net ILLUM_GND: no longer LED3.1 (K), LED6.1 (K), LED9.1 (K)
- net BL1_1 renamed +5V_PNL
- net +5V_PNL: now also J1.26, LED2.2 (A), LED3.2 (A), LED5.2 (A), LED6.2 (A), LED8.2 (A), LED9.2 (A), C1.1, C2.1, C3.1, LED10.2 (A), LED11.2 (A), LED12.2 (A), LED13.2 (A), LED14.2 (A), LED15.2 (A), LED16.2 (A), LED17.2 (A), LED18.2 (A), LED19.2 (A), LED20.2 (A), LED21.2 (A), LED22.2 (A), LED23.2 (A), LED24.2 (A), LED25.2 (A), LED26.2 (A), LED27.2 (A), LED28.2 (A), LED29.2 (A), LED30.2 (A), LED31.2 (A), LED32.2 (A), LED33.2 (A), LED34.2 (A), LED35.2 (A), U2.41 (VCC); no longer R1.2
- net BL1_2 renamed LK1
- net LK1: now also U2.47 (OUT1); no longer LED2.2 (A)
- net BL1_3 renamed LK2
- net LK2: now also U2.48 (OUT2); no longer LED3.2 (A)
- net BL2_2 renamed LK4
- net LK4: now also U2.2 (OUT4); no longer LED5.2 (A)
- net BL2_3 renamed LK5
- net LK5: now also U2.3 (OUT5); no longer LED6.2 (A)
- net BL3_2 renamed LK7
- net LK7: now also U2.6 (OUT7); no longer LED8.2 (A)
- net BL3_3 renamed LK8
- net LK8: now also U2.7 (OUT8); no longer LED9.2 (A)
- new net LED_REXT: R1.1, U2.44 (R_EXT)
- new net LED_SDB: R2.1, U2.39 (SDB)
- new net LF1: LED10.1 (K), U2.9 (OUT10)
- new net LF2: LED11.1 (K), U2.10 (OUT11)
- new net LF3: LED12.1 (K), U2.11 (OUT12)
- new net LF4: LED13.1 (K), U2.12 (OUT13)
- new net LF5: LED14.1 (K), U2.13 (OUT14)
- new net LF6: LED15.1 (K), U2.14 (OUT15)
- new net LF7: LED16.1 (K), U2.15 (OUT16)
- new net LK3: LED3.1 (K), U2.1 (OUT3)
- new net LK6: LED6.1 (K), U2.5 (OUT6)
- new net LK9: LED9.1 (K), U2.8 (OUT9)
- new net LSD1: LED24.1 (K), U2.25 (OUT24)
- new net LSD2: LED25.1 (K), U2.26 (OUT25)
- new net LSD3: LED26.1 (K), U2.27 (OUT26)
- new net LSD4: LED27.1 (K), U2.28 (OUT27)
- new net LSD5: LED28.1 (K), U2.29 (OUT28)
- new net LSD6: LED29.1 (K), U2.30 (OUT29)
- new net LSP1: LED30.1 (K), U2.31 (OUT30)
- new net LSP2: LED31.1 (K), U2.32 (OUT31)
- new net LSP3: LED32.1 (K), U2.34 (OUT32)
- new net LSP4: LED33.1 (K), U2.35 (OUT33)
- new net LSP5: LED34.1 (K), U2.36 (OUT34)
- new net LSP6: LED35.1 (K), U2.37 (OUT35)
- new net LT1: LED17.1 (K), U2.16 (OUT17)
- new net LT2: LED18.1 (K), U2.17 (OUT18)
- new net LT3: LED19.1 (K), U2.20 (OUT19)
- new net LT4: LED20.1 (K), U2.21 (OUT20)
- new net LT5: LED21.1 (K), U2.22 (OUT21)
- new net LT6: LED22.1 (K), U2.23 (OUT22)
- new net LT7: LED23.1 (K), U2.24 (OUT23)
- new net PNL_SCL: J1.24, U2.46 (SCL)
- new net PNL_SDA: J1.22, U2.45 (SDA)
- new net SPARE: J1.25, TP1.1
- no-connect marks 0 -> 1
Other:
- note added: "- ILLUM_12V / ILLUM_GND (J2, DNP) feed only the style-(b) light rings: J2 is fitted with SWB1-9 if 03.14 is (b)."
- note added: "- The lights (D-458): LED colours, the 7.6 mA ceiling (R1) and the window positions are confirm until LP20 and the bench."
- note added: "0x74 / 0x75 (expanders, SN17) and 0x48 (ADC, SN29) are the carrier's. +5V_PNL from ribbon pin 26 (PTC F1 on the carrier)."
- note added: "22 kHz PWM (register 4Bh) keeps the ceramic caps silent (p.12). SDB held high by R2: powers up blank (p.9)."
- note added: "A key's LED sits by its key; each knob has an arc of LEDs over it: fan and temperature 7 steps, each seat cool 3-2-1 | OFF | heat 1-2-3. Windows: panel/README.md. Colours and currents are LP20's and the bench's - confirm."
- note added: "Dimming (D-462): the DCU scales every channel's PWM to the dash dimmer level and writes the update register 25h;"
- note added: "IS31FL3236A-TQLS4 (eTQFP-48, -40 to +125 C) on the back, I2C 0x3C (AD to GND), on the DCU's bus:"
- note added: "LIGHT DRIVER (D-458, D-462)"
- note added: "LIGHTS (D-458) - 35 LEDs on the faceplate side, anode +5V_PNL, cathode to one IS31FL3236A channel each (OUT1-OUT35, OUT36 spare)"
- note added: "OUT1-9 keys in 0x400 bit order, OUT10-16 fan, OUT17-23 temperature, OUT24-29 driver seat, OUT30-35 passenger seat, OUT36 open."
- note added: "One channel per LED; R1 10k sets IMAX = 58.5 x 1.3 V / 10k = 7.6 mA (p.11); 256 PWM steps per channel."
- note added: "Ribbon to the DCU - 26-way 2.54 mm IDC box header, keyed, panel end (P157, panel_ribbon, D-458): 1-20 as before, 21 GND, 22 PNL_SDA, 23 GND, 24 PNL_SCL, 25 SPARE, 26 +5V_PNL"
- note added: "illumination in (DNP) - its own lead from L3-S1 8 (DV53, PV94): only for the style-(b) rings; the panel LEDs dim over I2C (D-462)"
- note removed: "- ILLUM_12V / ILLUM_GND feed only DNP parts: the backlight and the (b) rings wait on 03.14 and 01.14."
- note removed: "- No indicator lamps: the ribbon has no conductor for them (a block)."
- note removed: "BACKLIGHT FOR KEY STYLE (a) - DNP: three strings of three LEDs off the illumination input, one string per matrix row"
- note removed: "LEDn sits beside key SWn under its cap. ~5 mA per string at 13.8 V with white LEDs (13.8 - 3 x 2.9 V) / 1k. Values, colour and whether the keys are backlit at all wait on 03.14 and 01.14 - confirm."
- note removed: "Ribbon to the DCU - 20-way 2.54 mm IDC box header, panel end (P157, panel_ribbon)"
- note removed: "illumination in - its own lead from L3-S1 8, dims with the dash (DV53, PV94): feeds the backlight below (DNP)"

Commit message: Electrical: the panel board redrawn to the ruled control set and the DCU sheet renamed to the ribbon; both packaged for the bench order with the upper board (Y20)
panel rev 0.04: 180 x 84.76 mm with the controls where the sketch puts them, a 4 x 3 matrix, one centre encoder with push, two seat encoders, DPDT sprung window switches, the screen header behind its window with a supply jumper, the LED driver with 24 LEDs, the 26-way ribbon and the 2 x 6 plate header; ERC 0, DRC and parity 0, check.py 79 checks 0 mismatches. The DCU carrier's ribbon nets renamed (sheet, symbol pins, board net names only; DRC and parity 0, check.py 163 / 0); check.py's panel and dcu entries follow the record. Found and recorded: the window switches must be double-pole, the screen a 3.3 V-bus module, the seat symbol cannot sit in the knob's centre without a hollow-shaft encoder. Gerbers, drills and BOMs for the panel and upper boards under fab/ for Y18; the climate-unit mock-up's ribbon header at the drawn 16.5 mm, rebuilt clear.

Co-Authored-By: Claude Fable 5.1 <noreply@anthropic.com>
Parts:
- removed D9: 1N4148W, Diode_SMD:D_SOD-123, symbol panel:D
- removed J2: illumination in, Connector_JST:JST_XH_B2B-XH-A_1x02_P2.50mm_Vertical, symbol panel:Conn_01x02
- removed LED25: driver seat cool 2 - confirm, LED_SMD:LED_0603_1608Metric, symbol panel:LED
- removed LED26: driver seat cool 1 - confirm, LED_SMD:LED_0603_1608Metric, symbol panel:LED
- removed LED27: driver seat heat 1 - confirm, LED_SMD:LED_0603_1608Metric, symbol panel:LED
- removed LED28: driver seat heat 2 - confirm, LED_SMD:LED_0603_1608Metric, symbol panel:LED
- removed LED29: driver seat heat 3 - confirm, LED_SMD:LED_0603_1608Metric, symbol panel:LED
- removed LED30: passenger seat cool 3 - confirm, LED_SMD:LED_0603_1608Metric, symbol panel:LED
- removed LED31: passenger seat cool 2 - confirm, LED_SMD:LED_0603_1608Metric, symbol panel:LED
- removed LED32: passenger seat cool 1 - confirm, LED_SMD:LED_0603_1608Metric, symbol panel:LED
- removed LED33: passenger seat heat 1 - confirm, LED_SMD:LED_0603_1608Metric, symbol panel:LED
- removed LED34: passenger seat heat 2 - confirm, LED_SMD:LED_0603_1608Metric, symbol panel:LED
- removed LED35: passenger seat heat 3 - confirm, LED_SMD:LED_0603_1608Metric, symbol panel:LED
- removed SW10: encoder - fan, panel:RotaryEncoder_Bourns_Vertical_PEC11R-4xxxF-Sxxxx, symbol panel:ENCODER_AB
- removed SW11: encoder - temperature, panel:RotaryEncoder_Bourns_Vertical_PEC11R-4xxxF-Sxxxx, symbol panel:ENCODER_AB
- removed SW12: encoder - driver seat, panel:RotaryEncoder_Bourns_Vertical_PEC11R-4xxxF-Sxxxx, symbol panel:ENCODER_AB
- removed SW13: encoder - passenger seat, panel:RotaryEncoder_Bourns_Vertical_PEC11R-4xxxF-Sxxxx, symbol panel:ENCODER_AB
- removed SW5: key - recirculate, Button_Switch_THT:SW_PUSH_6mm_H13mm, symbol panel:SW_Push
- removed SW6: key - window DRV up, Button_Switch_THT:SW_PUSH_6mm_H13mm, symbol panel:SW_Push
- removed SW7: key - window DRV down, Button_Switch_THT:SW_PUSH_6mm_H13mm, symbol panel:SW_Push
- removed SW8: key - window PASS up, Button_Switch_THT:SW_PUSH_6mm_H13mm, symbol panel:SW_Push
- removed SW9: key - window PASS down, Button_Switch_THT:SW_PUSH_6mm_H13mm, symbol panel:SW_Push
- removed SWB1: key (b) - defog, Connector_JST:JST_XH_B4B-XH-A_1x04_P2.50mm_Vertical, symbol panel:SW_Push_LED
- removed SWB2: key (b) - hatch release, Connector_JST:JST_XH_B4B-XH-A_1x04_P2.50mm_Vertical, symbol panel:SW_Push_LED
- removed SWB3: key (b) - fuel-door release, Connector_JST:JST_XH_B4B-XH-A_1x04_P2.50mm_Vertical, symbol panel:SW_Push_LED
- removed SWB4: key (b) - HVAC mode, Connector_JST:JST_XH_B4B-XH-A_1x04_P2.50mm_Vertical, symbol panel:SW_Push_LED
- removed SWB5: key (b) - recirculate, Connector_JST:JST_XH_B4B-XH-A_1x04_P2.50mm_Vertical, symbol panel:SW_Push_LED
- removed SWB6: key (b) - window DRV up, Connector_JST:JST_XH_B4B-XH-A_1x04_P2.50mm_Vertical, symbol panel:SW_Push_LED
- removed SWB7: key (b) - window DRV down, Connector_JST:JST_XH_B4B-XH-A_1x04_P2.50mm_Vertical, symbol panel:SW_Push_LED
- removed SWB8: key (b) - window PASS up, Connector_JST:JST_XH_B4B-XH-A_1x04_P2.50mm_Vertical, symbol panel:SW_Push_LED
- removed SWB9: key (b) - window PASS down, Connector_JST:JST_XH_B4B-XH-A_1x04_P2.50mm_Vertical, symbol panel:SW_Push_LED
- removed U1: thumbstick - not chosen (P156), panel:Thumbstick_P156_Placeholder_2x04_P2.54mm, symbol panel:THUMBSTICK_2AX
- added J2: screen module I2C 4-pin, Connector_PinHeader_2.54mm:PinHeader_1x04_P2.54mm_Vertical, symbol panel:Conn_01x04
- added J3: plate header 2x6 IDC, keyed (DP-DCU-E 1-12), Connector_IDC:IDC-Header_2x06_P2.54mm_Vertical, symbol panel:Conn_02x06
- added JP1: screen supply 1-2 +5V_PNL / 2-3 +3V3, Jumper:SolderJumper-3_P1.3mm_Open_RoundedPad1.0x1.5mm, symbol panel:SolderJumper_3_Open
- added SW5: window DRV, panel:Toggle_DPDT_SubMini_2x3_P2.54mm, symbol panel:TOGGLE_DPDT_MOM
- added SW6: window PASS, panel:Toggle_DPDT_SubMini_2x3_P2.54mm, symbol panel:TOGGLE_DPDT_MOM
- added SW7: encoder - centre, panel:RotaryEncoder_Bourns_Vertical_PEC11R-4xxxF-Sxxxx, symbol panel:ENCODER_AB_SW
- added SW8: encoder - driver seat, panel:RotaryEncoder_Bourns_Vertical_PEC11R-4xxxF-Sxxxx, symbol panel:ENCODER_AB
- added SW9: encoder - passenger seat, panel:RotaryEncoder_Bourns_Vertical_PEC11R-4xxxF-Sxxxx, symbol panel:ENCODER_AB
- C1: value 10u 16V X7R - confirm -> 10uF 16V X7R; Confirm bulk at the ribbon entry for the LEDs' PWM current; X7R 080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 -> at J1 pin 26, for the LEDs' PWM current - part number confi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
- C2: value 1u -> 1uF; Confirm at U2 VCC (p.1 typical application) -> at U2 VCC - part number confirm (P192)
- C3: value 100n -> 100nF; Confirm at U2 VCC (p.1 typical application) -> at U2 VCC - part number confirm (P192)
- J1: Confirm 2 x 13 shrouded box header, 2.54 mm, keyed: the IDC plug go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 -> keyed shrouded box header, the part bought confirm (P157); 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
- LED1: value key light defog - confirm -> key light rear defog; footprint LED_SMD:LED_1206_3216Metric -> LED_SMD:LED_0603_1608Metric; Confirm by key SW1, under a faceplate window (panel/README.md); col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 -> 0603; colour per LP20 (P192), brightness on the bench - con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
- LED10: value fan level 1 - confirm -> window symbol PASS; Confirm fan knob arc, step 1 of 7 anticlockwise to clockwise; colou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 -> 0603; colour per LP20 (P192), brightness on the bench - con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
- LED11: value fan level 2 - confirm -> seat symbol DRV; Confirm fan knob arc, step 2 of 7 anticlockwise to clockwise; colou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 -> 0603; colour per LP20 (P192), brightness on the bench - con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
- LED12: value fan level 3 - confirm -> seat symbol PASS; Confirm fan knob arc, step 3 of 7 anticlockwise to clockwise; colou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 -> 0603; colour per LP20 (P192), brightness on the bench - con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
- LED13: value fan level 4 - confirm -> driver seat cool 3; Confirm fan knob arc, step 4 of 7 anticlockwise to clockwise; colou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 -> 0603; colour per LP20 (P192), brightness on the bench - con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
- LED14: value fan level 5 - confirm -> driver seat cool 2; Confirm fan knob arc, step 5 of 7 anticlockwise to clockwise; colou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 -> 0603; colour per LP20 (P192), brightness on the bench - con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
- LED15: value fan level 6 - confirm -> driver seat cool 1; Confirm fan knob arc, step 6 of 7 anticlockwise to clockwise; colou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 -> 0603; colour per LP20 (P192), brightness on the bench - con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
- LED16: value fan level 7 - confirm -> driver seat heat 1; Confirm fan knob arc, step 7 of 7 anticlockwise to clockwise; colou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 -> 0603; colour per LP20 (P192), brightness on the bench - con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
- LED17: value temperature level 1 - confirm -> driver seat heat 2; Confirm temperature knob arc, step 1 of 7 anticlockwise to clockwis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 -> 0603; colour per LP20 (P192), brightness on the bench - con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
- LED18: value temperature level 2 - confirm -> driver seat heat 3; Confirm temperature knob arc, step 2 of 7 anticlockwise to clockwis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 -> 0603; colour per LP20 (P192), brightness on the bench - con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
- LED19: value temperature level 3 - confirm -> passenger seat cool 3; Confirm temperature knob arc, step 3 of 7 anticlockwise to clockwis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 -> 0603; colour per LP20 (P192), brightness on the bench - con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
- LED2: value key light hatch release - confirm -> key light HVAC mode; footprint LED_SMD:LED_1206_3216Metric -> LED_SMD:LED_0603_1608Metric; Confirm by key SW2, under a faceplate window (panel/README.md); col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 -> 0603; colour per LP20 (P192), brightness on the bench - con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
- LED20: value temperature level 4 - confirm -> passenger seat cool 2; Confirm temperature knob arc, step 4 of 7 anticlockwise to clockwis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 -> 0603; colour per LP20 (P192), brightness on the bench - con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
- LED21: value temperature level 5 - confirm -> passenger seat cool 1; Confirm temperature knob arc, step 5 of 7 anticlockwise to clockwis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 -> 0603; colour per LP20 (P192), brightness on the bench - con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
- LED22: value temperature level 6 - confirm -> passenger seat heat 1; Confirm temperature knob arc, step 6 of 7 anticlockwise to clockwis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 -> 0603; colour per LP20 (P192), brightness on the bench - con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
- LED23: value temperature level 7 - confirm -> passenger seat heat 2; Confirm temperature knob arc, step 7 of 7 anticlockwise to clockwis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 -> 0603; colour per LP20 (P192), brightness on the bench - con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
- LED24: value driver seat cool 3 - confirm -> passenger seat heat 3; Confirm driver seat knob arc: cool 3-1 anticlockwise of OFF, heat 1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 -> 0603; colour per LP20 (P192), brightness on the bench - con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
- LED3: value key light fuel-door release - confirm -> key light recirculate; footprint LED_SMD:LED_1206_3216Metric -> LED_SMD:LED_0603_1608Metric; Confirm by key SW3, under a faceplate window (panel/README.md); col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 -> 0603; colour per LP20 (P192), brightness on the bench - con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
- LED4: value key light HVAC mode - confirm -> key light mirror defog; footprint LED_SMD:LED_1206_3216Metric -> LED_SMD:LED_0603_1608Metric; Confirm by key SW4, under a faceplate window (panel/README.md); col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 -> 0603; colour per LP20 (P192), brightness on the bench - con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
- LED5: value key light recirculate - confirm -> knob ring 1; footprint LED_SMD:LED_1206_3216Metric -> LED_SMD:LED_0603_1608Metric; Confirm by key SW5, under a faceplate window (panel/README.md); col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 -> 0603; colour per LP20 (P192), brightness on the bench - con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
- LED6: value key light window DRV up - confirm -> knob ring 2; footprint LED_SMD:LED_1206_3216Metric -> LED_SMD:LED_0603_1608Metric; Confirm by key SW6, under a faceplate window (panel/README.md); col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 -> 0603; colour per LP20 (P192), brightness on the bench - con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
- LED7: value key light window DRV down - confirm -> knob ring 3; footprint LED_SMD:LED_1206_3216Metric -> LED_SMD:LED_0603_1608Metric; Confirm by key SW7, under a faceplate window (panel/README.md); col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 -> 0603; colour per LP20 (P192), brightness on the bench - con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
- LED8: value key light window PASS up - confirm -> knob ring 4; footprint LED_SMD:LED_1206_3216Metric -> LED_SMD:LED_0603_1608Metric; Confirm by key SW8, under a faceplate window (panel/README.md); col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 -> 0603; colour per LP20 (P192), brightness on the bench - con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
- LED9: value key light window PASS down - confirm -> window symbol DRV; footprint LED_SMD:LED_1206_3216Metric -> LED_SMD:LED_0603_1608Metric; Confirm by key SW9, under a faceplate window (panel/README.md); col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 -> 0603; colour per LP20 (P192), brightness on the bench - con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
- R1: Confirm R_EXT: IMAX = 58.5 x 1.3 V / R (p.11) = 7.6 mA per channel;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 -> IMAX 7.6 mA per channel (p.11) - part number confirm (P192)
- R2: Confirm SDB pull-up: enabled whenever +5V_PNL is up; registers powe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 -> SDB held high: on and blank until written - part number con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
- SW1: value key - defog -> key - rear defog; Confirm 03.14 (a): low-travel board switch under a faceplate cap, 6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 -> 6 x 6 mm THT tactile, 13 mm actuator under the faceplate's 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
- SW2: value key - hatch release -> key - HVAC mode; Confirm 03.14 (a): low-travel board switch under a faceplate cap, 6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 -> 6 x 6 mm THT tactile, 13 mm actuator under the faceplate's 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
- SW3: value key - fuel-door release -> key - recirculate; Confirm 03.14 (a): low-travel board switch under a faceplate cap, 6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 -> 6 x 6 mm THT tactile, 13 mm actuator under the faceplate's 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
- SW4: value key - HVAC mode -> key - mirror defog; Confirm 03.14 (a): low-travel board switch under a faceplate cap, 6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 -> 6 x 6 mm THT tactile, 13 mm actuator under the faceplate's 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
- TP1: Confirm ribbon pin 25 (SPARE): wired end to end so a later line needs no new cable -> ribbon pin 25 (SPARE): wired end to end so a later line needs no new cable (D-458)
- U2: Confirm Lumissil IS31FL3236A Rev. I: eTQFP-48 pinout p.2-3, land pa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 -> Lumissil IS31FL3236A-TQLS4, eTQFP-48 (P192); KiCad TQFP-48 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
Connections:
- net +3V3: now also J3.7, JP1.3
- net +5V_PNL: now also R2.1, J3.12, JP1.1; no longer R2.2
- net AGND: now also J3.8
- net COL1: now also SW1.2, SW2.2, SW4.2, SW5.4 (DN_2); no longer SW1.1, SW4.1
- net COL2: now also SW3.2, J3.2, SW6.3 (UP_1); no longer SW2.1
- net COL3: now also J3.3, SW5.3 (UP_1), SW6.4 (DN_2); no longer SW3.1
- net ENC_SEAT_DRV_A: now also SW8.1 (A)
- net ENC_SEAT_DRV_B: now also SW8.3 (B)
- net ENC_SEAT_PASS_A: now also SW9.1 (A)
- net ENC_SEAT_PASS_B: now also SW9.3 (B)
- net GND: now also J2.1 (Pin_1), J3.11, SW7.2 (C), SW7.S2, SW8.2 (C), SW9.2 (C)
- net JOY_PRESS: now also J3.6
- net JOY_X: now also J3.4
- net JOY_Y: now also J3.5
- net LED_SDB: now also R2.2; no longer R2.1
- net LK1: now also U2.3 (OUT5); no longer U2.47 (OUT1)
- net LK2: now also U2.6 (OUT7); no longer U2.48 (OUT2)
- net LK3: now also U2.31 (OUT30); no longer U2.1 (OUT3)
- net LK4: now also U2.35 (OUT33); no longer U2.2 (OUT4)
- net LSD1: now also LED13.1 (K), U2.9 (OUT10); no longer LED24.1 (K), U2.25 (OUT24)
- net LSD2: now also LED14.1 (K), U2.12 (OUT13); no longer U2.26 (OUT25)
- net LSD3: now also LED15.1 (K), U2.16 (OUT17); no longer U2.27 (OUT26)
- net LSD4: now also LED16.1 (K), U2.13 (OUT14); no longer U2.28 (OUT27)
- net LSD5: now also LED17.1 (K), U2.10 (OUT11); no longer U2.29 (OUT28)
- net LSD6: now also LED18.1 (K), U2.8 (OUT9); no longer U2.30 (OUT29)
- net LSP1: now also LED19.1 (K), U2.30 (OUT29); no longer U2.31 (OUT30)
- net LSP2: now also LED20.1 (K), U2.27 (OUT26); no longer U2.32 (OUT31)
- net LSP3: now also LED21.1 (K), U2.24 (OUT23); no longer U2.34 (OUT32)
- net LSP4: now also LED22.1 (K), U2.22 (OUT21); no longer U2.35 (OUT33)
- net LSP5: now also LED23.1 (K), U2.26 (OUT25); no longer U2.36 (OUT34)
- net LSP6: now also LED24.1 (K), U2.28 (OUT27); no longer U2.37 (OUT35)
- net PNL_SCL: now also J2.3 (Pin_3), J3.10
- net PNL_SDA: now also J2.4 (Pin_4), J3.9
- net ROW1: now also J3.1; no longer D2.1 (K), D3.1 (K)
- net ROW2: now also D2.1 (K), D3.1 (K); no longer D5.1 (K), D6.1 (K)
- net ROW3: now also D5.1 (K), D6.1 (K); no longer D8.1 (K)
- net ENC_FAN_A renamed ENC_CENTRE_A
- net ENC_CENTRE_A: now also SW7.1 (A)
- net ENC_FAN_B renamed ENC_CENTRE_B
- net ENC_CENTRE_B: now also SW7.3 (B)
- net ENC_TEMP_A renamed ENC_CENTRE_PUSH
- net ENC_CENTRE_PUSH: now also SW7.S1
- net ENC_TEMP_B renamed ROW4
- net ROW4: now also D8.1 (K)
- net K1_11: no longer names the net of D1.2 (A)
- net K1_11: now also SW1.1; no longer SW1.2
- net K2_12: no longer names the net of D2.2 (A)
- net K2_12: now also SW2.1; no longer SW2.2
- net K3_13: no longer names the net of D3.2 (A)
- net K3_13: now also SW3.1; no longer SW3.2
- net K4_21: no longer names the net of D4.2 (A)
- net K4_21: now also SW5.2 (COM_1); no longer SW4.2
- net K5_22: no longer names the net of D5.2 (A)
- net K5_22: now also SW5.5 (COM_2)
- net K6_23: no longer names the net of D6.2 (A)
- net K6_23: now also SW6.2 (COM_1)
- net K7_31: no longer names the net of D7.2 (A)
- net K7_31: now also SW6.5 (COM_2)
- net K8_32: no longer names the net of D8.2 (A)
- net K8_32: now also SW4.1
- net LF1 renamed LW2
- net LW2: now also U2.23 (OUT22); no longer U2.9 (OUT10)
- net LF2 renamed LS1
- net LS1: now also U2.17 (OUT18); no longer U2.10 (OUT11)
- net LF3: no longer names the net of U2.11 (OUT12)
- net LF3: no longer LED12.1 (K)
- removed net LF4: LED13.1 (K), U2.12 (OUT13)
- removed net LF5: LED14.1 (K), U2.13 (OUT14)
- net LF6 renamed LW1
- net LW1: now also LED9.1 (K); no longer LED15.1 (K)
- net LF7: no longer names the net of U2.15 (OUT16)
- net LF7: no longer LED16.1 (K)
- net LK5 renamed LR1
- net LR1: now also U2.5 (OUT6); no longer U2.3 (OUT5)
- net LK6 renamed LR2
- net LR2: now also U2.32 (OUT31); no longer U2.5 (OUT6)
- net LK7 renamed LR3
- net LR3: now also U2.36 (OUT34); no longer U2.6 (OUT7)
- net LK8: no longer names the net of U2.7 (OUT8)
- net LK8: no longer LED8.1 (K)
- removed net LK9: LED9.1 (K), U2.8 (OUT9)
- removed net LT1: LED17.1 (K), U2.16 (OUT17)
- removed net LT2: LED18.1 (K), U2.17 (OUT18)
- net LT3 renamed LS2
- net LS2: now also LED12.1 (K); no longer LED19.1 (K)
- net LT4: no longer names the net of U2.21 (OUT20)
- net LT4: no longer LED20.1 (K)
- removed net LT5: LED21.1 (K), U2.22 (OUT21)
- removed net LT6: LED22.1 (K), U2.23 (OUT22)
- removed net LT7: LED23.1 (K), U2.24 (OUT23)
- new net LR4: LED8.1 (K), U2.1 (OUT3)
- new net SCR_VCC: J2.2 (Pin_2), JP1.2
- no-connect marks 1 -> 16
Other:
- note added: "Centre: temperature; a push sets fan speed until it rests; fan mode after the fan-mode key (I-001)."
- note added: "HVAC mode: ROW2 / COL1"
- note added: "Headlight-only lights (the ring, the window and seat symbols) and state lights (the key symbols, the seat arcs) differ only in firmware (I-004)."
- note added: "J1: the 26-way ribbon to the DCU carrier's J4, pinned as panel_ribbon (P157, D-458, D-492)."
- note added: "J2 takes the module's own 4-pin header, GND - VCC - SCL - SDA (the common order, confirm on the module bought)."
- note added: "J3: the left plate's twelve lines, DP-DCU-E 1-12 pin for pin, by a lead to the upper board's J8 (D-492, Y21)."
- note added: "JP1 picks its supply: 1-2 +5V_PNL (the record: +3V3 feeds only the stick) or 2-3 +3V3. A module whose I2C pull-ups go"
- note added: "KEYS - 4 x 3 matrix, one 1N4148W per key, cathode to the row: a driven-low row pulls its column low (D-492)"
- note added: "KNOBS - detented quadrature encoders, common to GND (D-355, D-492)"
- note added: "LIGHTS - IS31FL3236A, I2C 0x3C (AD to GND), 36 constant-current sinks; each LED anode on +5V_PNL (D-458, D-492)"
- note added: "POWER - ribbon only: +5V_PNL behind the carrier's PTC F1, +3V3 for the stick (D-458, D-492)"
- note added: "R1 10 k sets IMAX = 58.5 x 1.3 V / 10 k = 7.6 mA (p.11); R2 100 k holds SDB high so the chip is on and blank until written."
- note added: "RIBBON AND PLATE HEADER"
- note added: "ROW1: rear defog (here) - hatch, fuel door (left plate, through J3 1-3) ROW2: HVAC mode - recirculate - window DRV up"
- note added: "ROW3: window DRV down - window PASS up - window PASS down ROW4: mirror defog - spare - spare"
- note added: "SCREEN - a 128 x 64-class I2C module on the panel bus (P201, D-492)"
- note added: "Seats: OFF in the middle, clockwise heat 1-3, anticlockwise cool 1-3 (D-073, I-003); no push."
- note added: "The window switches are centre-sprung DPDT: one pole per direction, so DRV up (ROW2/COL3) and DRV down (ROW3/COL1)"
- note added: "are two independent keys; an SPDT's single common cannot reach two rows and two columns without a phantom key."
- note added: "mirror defog: ROW4 / COL1"
- note added: "rear defog: ROW1 / COL1"
- note added: "recirculate: ROW2 / COL2"
- note added: "to its VCC must not run at 5 V on this bus (the Teensy's pins are 3.3 V): bridge 2-3 or remove them - confirm (P201)."
- note added: "window DRV up: ROW2 / COL3 (pole 1) down: ROW3 / COL1 (pole 2)"
- note added: "window PASS up: ROW3 / COL2 (pole 1) down: ROW3 / COL3 (pole 2)"
- note removed: "- AGND is its own ribbon conductor (pin 20), joined to GND only at the DCU carrier."
- note removed: "- Both key styles are drawn (SWn fitted, SWBn DNP); encoder and stick parts are confirm until V-113 and LP20."
- note removed: "- ILLUM_12V / ILLUM_GND (J2, DNP) feed only the style-(b) light rings: J2 is fitted with SWB1-9 if 03.14 is (b)."
- note removed: "- The lights (D-458): LED colours, the 7.6 mA ceiling (R1) and the window positions are confirm until LP20 and the bench."
- note removed: "0x74 / 0x75 (expanders, SN17) and 0x48 (ADC, SN29) are the carrier's. +5V_PNL from ribbon pin 26 (PTC F1 on the carrier)."
- note removed: "22 kHz PWM (register 4Bh) keeps the ceramic caps silent (p.12). SDB held high by R2: powers up blank (p.9)."
- note removed: "A key's LED sits by its key; each knob has an arc of LEDs over it: fan and temperature 7 steps, each seat cool 3-2-1 | OFF | heat 1-2-3. Windows: panel/README.md. Colours and currents are LP20's and the bench's - confirm."
- note removed: "Dimming (D-462): the DCU scales every channel's PWM to the dash dimmer level and writes the update register 25h;"
- note removed: "ENCODERS - common to GND, pull-ups on the DCU (SN20)"
- note removed: "Each SWBn sits in parallel with SWn on the same column and diode: fit SW1-SW9 (style a, recommended) or SWB1-SWB9 (style b), never both. Ring LED 3-4 across the illumination input; a 12 V ring with its own resistor - confirm."
- note removed: "IS31FL3236A-TQLS4 (eTQFP-48, -40 to +125 C) on the back, I2C 0x3C (AD to GND), on the DCU's bus:"
- note removed: "KEY STYLE (b) - ALTERNATES, DNP: a 12-16 mm round button with a light ring, wired to the board on a 4-way JST-XH (luxury 03.14 open)"
- note removed: "KEYS - 3 x 3 matrix, one diode per key, anode toward the column: a driven-low row pulls its column low (D-380)"
- note removed: "LIGHT DRIVER (D-458, D-462)"
- note removed: "LIGHTS (D-458) - 35 LEDs on the faceplate side, anode +5V_PNL, cathode to one IS31FL3236A channel each (OUT1-OUT35, OUT36 spare)"
- note removed: "OUT1-9 keys in 0x400 bit order, OUT10-16 fan, OUT17-23 temperature, OUT24-29 driver seat, OUT30-35 passenger seat, OUT36 open."
- note removed: "One channel per LED; R1 10k sets IMAX = 58.5 x 1.3 V / 10k = 7.6 mA (p.11); 256 PWM steps per channel."
- note removed: "PWR_FLAGs"
- note removed: "RIBBON"
- note removed: "ROW1 x COL1 defog"
- note removed: "ROW1 x COL2 hatch release"
- note removed: "ROW1 x COL3 fuel-door release"
- note removed: "ROW2 x COL1 HVAC mode"
- note removed: "ROW2 x COL2 recirculate"
- note removed: "ROW2 x COL3 window DRV up"
- note removed: "ROW3 x COL1 window DRV down"
- note removed: "ROW3 x COL2 window PASS up"
- note removed: "ROW3 x COL3 window PASS down"
- note removed: "Ribbon to the DCU - 26-way 2.54 mm IDC box header, keyed, panel end (P157, panel_ribbon, D-458): 1-20 as before, 21 GND, 22 PNL_SDA, 23 GND, 24 PNL_SCL, 25 SPARE, 26 +5V_PNL"
- note removed: "THUMBSTICK AND ILLUMINATION"
- note removed: "WHAT THIS SHEET DOES NOT KNOW (R11)"
- note removed: "driver seat: cw heat 1-3, ccw cool 1-3"
- note removed: "fan"
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