File: 02-PROJECTS/01-electrical/00-design/control-unit/cad/panel/panel.kicad_sch (KiCad schematic)
At the start: 52 parts, among them J1 panel ribbon 2x13 IDC, keyed, J2 screen module I2C 4-pin, J3 plate header 2x6 IDC, keyed (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, SW1 key - rear defog, SW2 key - HVAC mode, SW3 key - recirculate, SW4 key - mirror defog, SW5 window DRV, SW6 window PASS, SW7 encoder - centre, SW8 encoder - driver seat, SW9 encoder - passenger seat, U2 IS31FL3236A-TQLS4

Commit message: Electrical: the carriers corrected before the order - six TVS diodes drawn backwards, the wake switch's pins swapped, an unconnected zener, the bulk capacitor's value (D-547)
Y42 done; Y44 (an independent read of the boards, and the gate drive of two P-FETs) holds the board order Y18. DU and CU carrier fab zips rebuilt; the earlier ones must not be ordered. The board check now holds transistors and diodes to their makers' pin-outs.

Co-Authored-By: Claude Opus 5.5 <noreply@anthropic.com>
Parts:
- SW1, SW2, SW3, SW4: Confirm 6 x 6 mm THT tactile, 13 mm actuator under the faceplate's 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 -> Same Sky TS02-66-130-BK-160-LCR-D (P155, luxury D-488): 6 x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
Changed lines of the file:
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@@
 		(property "Footprint" "Button_Switch_THT:SW_PUSH_6mm_H13mm" (at 213.36 55.88 0) (effects (font (size 1.1 1.1)) (hide yes)))
 		(property "Datasheet" "" (at 213.36 55.88 0) (effects (font (size 1.1 1.1)) (hide yes)))
-		(property "Confirm" "6 x 6 mm THT tactile, 13 mm actuator under the faceplate's cap (luxury D-488, P155); actuator height confirm (LP20)" (at 213.36 55.88 0) (effects (font (size 1.1 1.1)) (hide yes)))
+		(property "Confirm" "Same Sky TS02-66-130-BK-160-LCR-D (P155, luxury D-488): 6 x 6 mm THT tactile, its top 13.0 mm above the board, 160 gf. The footprint is the maker's drawing rev 1.03: 6.5 x 4.5 mm, four 1.0 mm holes, pins 1-2 and 3-4 joined. The mock-up puts the cap's front 13 mm from the board (8 + 3 + 2): the cap's own top adds to that, or the 12.0 mm TS02-66-120-BK-160-LCR-D leaves it 1 mm - confirm with the cap (LP20)" (at 213.36 55.88 0) (effects (font (size 1.1 1.1)) (hide yes)))
 		(pin "1")
 		(pin "2")
@@
 		(property "Footprint" "Button_Switch_THT:SW_PUSH_6mm_H13mm" (at 213.36 68.58 0) (effects (font (size 1.1 1.1)) (hide yes)))
 		(property "Datasheet" "" (at 213.36 68.58 0) (effects (font (size 1.1 1.1)) (hide yes)))
-		(property "Confirm" "6 x 6 mm THT tactile, 13 mm actuator under the faceplate's cap (luxury D-488, P155); actuator height confirm (LP20)" (at 213.36 68.58 0) (effects (font (size 1.1 1.1)) (hide yes)))
+		(property "Confirm" "Same Sky TS02-66-130-BK-160-LCR-D (P155, luxury D-488): 6 x 6 mm THT tactile, its top 13.0 mm above the board, 160 gf. The footprint is the maker's drawing rev 1.03: 6.5 x 4.5 mm, four 1.0 mm holes, pins 1-2 and 3-4 joined. The mock-up puts the cap's front 13 mm from the board (8 + 3 + 2): the cap's own top adds to that, or the 12.0 mm TS02-66-120-BK-160-LCR-D leaves it 1 mm - confirm with the cap (LP20)" (at 213.36 68.58 0) (effects (font (size 1.1 1.1)) (hide yes)))
 		(pin "1")
 		(pin "2")
@@
 		(property "Footprint" "Button_Switch_THT:SW_PUSH_6mm_H13mm" (at 213.36 81.28 0) (effects (font (size 1.1 1.1)) (hide yes)))
 		(property "Datasheet" "" (at 213.36 81.28 0) (effects (font (size 1.1 1.1)) (hide yes)))
-		(property "Confirm" "6 x 6 mm THT tactile, 13 mm actuator under the faceplate's cap (luxury D-488, P155); actuator height confirm (LP20)" (at 213.36 81.28 0) (effects (font (size 1.1 1.1)) (hide yes)))
+		(property "Confirm" "Same Sky TS02-66-130-BK-160-LCR-D (P155, luxury D-488): 6 x 6 mm THT tactile, its top 13.0 mm above the board, 160 gf. The footprint is the maker's drawing rev 1.03: 6.5 x 4.5 mm, four 1.0 mm holes, pins 1-2 and 3-4 joined. The mock-up puts the cap's front 13 mm from the board (8 + 3 + 2): the cap's own top adds to that, or the 12.0 mm TS02-66-120-BK-160-LCR-D leaves it 1 mm - confirm with the cap (LP20)" (at 213.36 81.28 0) (effects (font (size 1.1 1.1)) (hide yes)))
 		(pin "1")
 		(pin "2")
@@
 		(property "Footprint" "Button_Switch_THT:SW_PUSH_6mm_H13mm" (at 213.36 93.98 0) (effects (font (size 1.1 1.1)) (hide yes)))
 		(property "Datasheet" "" (at 213.36 93.98 0) (effects (font (size 1.1 1.1)) (hide yes)))
-		(property "Confirm" "6 x 6 mm THT tactile, 13 mm actuator under the faceplate's cap (luxury D-488, P155); actuator height confirm (LP20)" (at 213.36 93.98 0) (effects (font (size 1.1 1.1)) (hide yes)))
+		(property "Confirm" "Same Sky TS02-66-130-BK-160-LCR-D (P155, luxury D-488): 6 x 6 mm THT tactile, its top 13.0 mm above the board, 160 gf. The footprint is the maker's drawing rev 1.03: 6.5 x 4.5 mm, four 1.0 mm holes, pins 1-2 and 3-4 joined. The mock-up puts the cap's front 13 mm from the board (8 + 3 + 2): the cap's own top adds to that, or the 12.0 mm TS02-66-120-BK-160-LCR-D leaves it 1 mm - confirm with the cap (LP20)" (at 213.36 93.98 0) (effects (font (size 1.1 1.1)) (hide yes)))
 		(pin "1")
 		(pin "2")
