File: 02-PROJECTS/01-electrical/00-design/display-unit/cad/icu-carrier/icu-carrier.kicad_pcb (KiCad board)
At the start: 2 copper layers, 110 x 80 mm, 118 parts, among them J1 DT13-06PA, J2 backlight out, J3 DT13-12PA, J4 ME817EV CN8 - 2x8 host header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, J5 Teensy 4.1 socket - 2 x 24 fe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, Q1 SQD50P06 class, >= 60 V, Q2 MMBT3904, Q3 DMG3415U class P-FET, SOT-23 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, Q4 MMBT3904, SW1 IC22, U1 LMR36015FSCQ-Q1, U3 TCAN1042HVDRQ1, U4 LM393, U5 74LVC1G17, U7 Adafruit 4517 LSM6DSOX+LIS3MD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, U8 XIAO ESP32C3 2x7 socket (Seee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

Commit message: Electrical: the carriers corrected before the order - six TVS diodes drawn backwards, the wake switch's pins swapped, an unconnected zener, the bulk capacitor's value (D-547)
Y42 done; Y44 (an independent read of the boards, and the gate drive of two P-FETs) holds the board order Y18. DU and CU carrier fab zips rebuilt; the earlier ones must not be ordered. The board check now holds transistors and diodes to their makers' pin-outs.

Co-Authored-By: Claude Opus 5.5 <noreply@anthropic.com>
Parts:
- C1: value 100u 63V -> 68u 63V
- turned D24 to -90 degrees
- turned D26 to -90 degrees
Connections:
- D20 pad 2: Net-(D20-A) -> Net-(D20-K)
- D20 pad 3: (no net) -> Net-(D20-K)
- D21 pad 3: Net-(D20-A) -> Net-(D20-K)
- D24 pad 1: GND -> +12V_LOGIC
- D24 pad 2: +12V_LOGIC -> GND
- D26 pad 1: GND -> +12V_BL
- D26 pad 2: +12V_BL -> GND
- R30 pad 1: Net-(D20-A) -> Net-(D20-K)
- R33 pad 2: Net-(D20-A) -> Net-(D20-K)
- U4 pad 3: Net-(D20-A) -> Net-(D20-K)
Routing:
- net Net-(D20-K): track 0.00 -> 20.9 mm
- net Net-(D20-A): track 18.8 -> 0.00 mm

Commit message: Electrical: the two P-FETs' gate drive brought down, the order text names the parts as they are (D-547)
CU Q3: R43 18 k, inside its gate limit at the 53 V clamp. DU Q1: R2 10 k, inside to 40 V on the rail; a gate zener for the clamp case is held for one fix pass with the independent review's findings (Y44). No fab file changed; the cart file follows. Y18's steps rebuilt.

Co-Authored-By: Claude Opus 5.5 <noreply@anthropic.com>
Parts:
- R2: value 1k -> 10k
Changed lines of the file:
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@@
 			)
 		)
-		(property "Value" "1k"
+		(property "Value" "10k"
 			(at 0 1.65 0)
 			(layer "F.Fab")

Commit message: Electrical: the independent read's findings fixed on the boards before the order, and the Display Unit's brake-warning input given its pull-up (D-549)
Y44 done; Y18 (the board order) opens. DU carrier rev 0.06: road-speed input IC08 re-laid, a 15 V gate zener and 4.7 k on the backlight switch, four vias at each backlight layer change, brake warning IC06 pulled up to 3V3 (found while the changes were read back - it could never have read high), tell-tale dividers 22 k, MMBT5551 and SL310A on the rails clamped at 53 V. CU carrier rev 0.07, values only: C27 100 nF, Q1 / Q2 SQ2364EES, Q4 MMBT5551, D1 SL310A. Panel: the encoders' lug slots to Bourns' layout. Two assembly drawings in each fab folder in place of silkscreen references.

ERC 0, DRC 0 / 0 / 0, check.py 0 mismatches on all five boards. The DU carrier's and the panel's fab zips are rebuilt under the same names; the CU carrier's and the upper board's are unchanged. Cart 98 lines. Record: icu_channels IC06 IC08 IC09 IC12 IC13, dcu_channels SN23 SN24, parts P106 P107 P147 P149 P169 P170 P203, Y18 / F3 / F5 briefs and steps. D-548's DT13 question is untouched (V-117).

Co-Authored-By: Claude Opus 5.5 <noreply@anthropic.com>
Parts:
- added D27: MM3Z15VT1G, Diode_SMD:D_SOD-323, B.Cu at (179.9, 78.5)
- D23, D25: value SS34 -> SL310A
- Q2: value MMBT3904 -> MMBT5551
- R16: value 47k -> 1k
- R2: value 10k -> 4.7k
- R21, R23, R25: value 47k -> 22k
- moved R17 8.23 mm to (136.0, 87.3), turned to 180 degrees
Connections:
- net Net-(Q1-G) renamed /BL_GATE
- net Net-(Q1-S) renamed /BL_FUSED
- D22 pad 3: /ICU_B8 -> /IC08_IN
- JP8B1 pad 1: /ICU_B8 -> GND
- R17 pad 2: GND -> +3V3
- R36 pad 1: Net-(JP8B1-Pad2) -> /ICU_B8
- R36 pad 2: /ICU_B8 -> /IC08_IN
- R37 pad 1: /ICU_B8 -> /IC08_IN
- R37 pad 2: GND -> Net-(JP8B1-Pad2)
- U5 pad 2: /ICU_B8 -> /IC08_IN
Routing:
- net /ICU_B8: track 62.4 -> 39.2 mm
- net /IC08_IN: track 0.00 -> 19.5 mm
- net Net-(JP8A1-Pad2): track 8.42 -> 4.46 mm
- net Net-(JP8B1-Pad2): track 5.67 -> 4.51 mm
- net /BL_FUSED: track 21.5 -> 22.5 mm
- net /BL_GATE: track 12.9 -> 13.7 mm, vias 2 -> 3
- net Net-(D25-A): vias 1 -> 4
- net +12V_BL_SW: vias 1 -> 4
- net +12V_BL: vias 2 -> 8

Commit message: Electrical: the ICU carrier drawn with one DRC13-24PA, the tach alone on pin 6; the board 110 x 84 (D-590, D-591, D-592)
Y63 done. J1 and J3 become one Deutsch DRC13-24PA (footprint from TE's drawing, TE's model in the
library and on the board), the board grows 4 mm at the connector edge, re-routed under the project's
own rules: ERC 0, DRC 0 with parity, check.py icu 105 / 0. The cavity map is permuted so the tach
(TACH_HV, 2.5 mm) has no live neighbour (D-592); every row, step and the engine handover follow.
Fab package, BOM, assembly, STEP, the DU mock-up (34 / 34) and the bench enclosure rebuilt; the DRC
family in the connector builder (the receptacle from TE's model); the scene re-exported. The record
files also carry Y62 / Y50's rows and block 01.60 (the next commit's boards).

Co-Authored-By: Claude Opus 5.5 <noreply@anthropic.com>
Parts:
- removed J3: DT13-12PA, icu-carrier:DT13-12PA
- J1: value DT13-06PA -> DRC13-24PA; footprint icu-carrier:DT13-06PA -> icu-carrier:DRC13-24PA
- moved J1 32.4 mm to (155.0, 54.1)
Connections:
- J1 pad 3: GND -> Net-(D25-A)
- J1 pad 6: Net-(D25-A) -> /ICU_B4
Routing:
- net GND: track 149.0 -> 1063.1 mm, vias 206 -> 231
- net /ICU_B2: track 5.86 -> 63.6 mm
- net /ICU_B1: track 36.9 -> 92.5 mm
- net /ICU_B3: track 38.6 -> 88.8 mm, vias 0 -> 1
- net /CAN2L_J: track 31.9 -> 79.6 mm, vias 2 -> 0
- net /CAN2H_J: track 28.3 -> 65.4 mm, vias 1 -> 4
- net /ICU_B7: track 63.0 -> 94.2 mm, vias 1 -> 2
- net /ICU_B12: track 41.8 -> 20.0 mm, vias 1 -> 0
- net Net-(D25-A): track 22.6 -> 7.19 mm, vias 4 -> 0
- net /IC14_IN: track 5.53 -> 17.9 mm
- net +3V3: track 335.6 -> 347.3 mm, vias 15 -> 13
- net /ICU_B5: track 10.4 -> 21.1 mm
- net /IC02_ADC: track 85.2 -> 93.7 mm
- net /IC06_DIG: track 20.8 -> 27.0 mm
- net /ICU_B11: track 30.6 -> 24.7 mm
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Other:
- board size 110 x 80 mm -> 110 x 84 mm
- board text added: "DP-ICU DRC13-24PA"
- board text added: "ICU carrier H-001 r0.07 - PROVISIONAL outline (C4, F11)"
- board text removed: "DP-ICU-A DT13-06PA"
- board text removed: "DP-ICU-B DT13-12PA"
- board text removed: "ICU carrier H-001 r0.03 - PROVISIONAL outline (C4, F11)"
