File: 02-PROJECTS/01-electrical/00-design/control-unit/control-unit-remote/cad/cur-board/cur-board.kicad_sch (KiCad schematic)
At the start: 26 parts, among them J1 plate cable header 2x6 shroud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, J2 wink lead header 1x5 (L3-S1 9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, J4 screen knob lead header (STEM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, SW1 key - hatch, SW2 key - fuel door, SW3 wink - left (P204), SW4 wink - right (P204), SW5 hazard - latching (P226), U1 IS31FL3218-QFLS2-TR

Commit message: 00-design: the CUR's CAD - board rev 1.00, the box mock-up, every CUR drawing current (D-615)
cur-board rev 1.00: 38.11 x 27.0, four layers, ERC 0, DRC 0 / 0 unconnected /
0 parity, check.py 26 checks 0 mismatches; fab package (16 files), assembly
drawings, BOM, schematic SVG. cur-assembly: shell 41.91 x 30.8 x 19.6, fit check
clear, self-test 13 of 13, four views. READMEs rewritten; plan sheets redrawn.

Co-Authored-By: Claude Opus 5.5 <noreply@anthropic.com>
Parts:
- removed D1, D2: 1N4148W, Diode_SMD:D_SOD-123, symbol cur-board:D
- removed J2: wink lead header 1x5 (L3-S1 9 / 10 / 11, commons,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, Connector_JST:JST_XH_B5B-XH-A_1x05_P2.50mm_Vertical, symbol cur-board:Conn_01x05
- removed J4: screen knob lead header (STEMMA QT, P219), Connector_JST:JST_SH_BM04B-SRSS-TB_1x04-1MP_P1.00mm_Vertical, symbol cur-board:Conn_01x04
- removed JS1: mirror stick (P156) - placeholder, cur-board:Thumbstick_P156_Placeholder_2x04_P2.54mm, symbol cur-board:THUMBSTICK_2AXIS_SW
- added C3: 100nF, Capacitor_SMD:C_0603_1608Metric, symbol cur-board:C
- added C4, C5: 1uF, Capacitor_SMD:C_0603_1608Metric, symbol cur-board:C
- added ENC1: screen knob - 9 mm encoder with push (P219), cur-board:ScreenKnob_Encoder9mm_Placeholder, symbol cur-board:RotaryEncoder_Switch
- added SW6: mirror control - 4 way + push (P156), cur-board:Thumbstick_SKRH_4Way_Push_Placeholder, symbol cur-board:SW_4WAY_PUSH
- added U2: PCA9555PW, Package_SO:TSSOP-24_4.4x7.8mm_P0.65mm, symbol cur-board:PCA9555PW
- added U3: AP2112K-3.3TRG1, Package_TO_SOT_SMD:SOT-23-5, symbol cur-board:AP2112K-3.3
- J1: value plate cable header 2x6 shrouded (DP-DCU-E 1-12, P200) -> pigtail solder pads 1x9 (DP-CUR 1-9); footprint Connector_IDC:IDC-Header_2x06_P2.54mm_Vertical -> cur-board:Pigtail_SolderPads_1x09_P2.54mm; symbol cur-board:Conn_02x06 -> cur-board:Conn_01x09; Confirm the cable's plate end (P200): pin n = DP-DCU-E n; IDC or cr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 -> the CUR's sealed pigtail (P200, D-615): nine 20 AWG conduct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
- LED1, LED2, LED3, LED4, LED6: Confirm colour, brightness and part number - confirm (I-006: the wink faces green; the rest LP20's) -> colour, brightness and part number - confirm (I-006: the wink faces green; the hazard red)
- LED5: value LED 0603 - mirror stick symbol (OUT13) -> LED 0603 - mirror symbol, in the control's well (OUT13); Confirm colour, brightness and part number - confirm (I-006: the wink faces green; the rest LP20's) -> colour, brightness and part number - confirm (I-006: the wink faces green; the hazard red)
- R1: Confirm R_EXT: IMAX = 58.5 x 1.3 V / 10k = 7.6 mA a channel (Lumissil p.10), the panel's D-458 current - 1 % -> R_EXT: IMAX = 58.5 x 1.3 V / 10k = 7.6 mA a channel (Lumissil p.10), the face board's current - 1 %
- R2: Confirm holds SDB high: the driver is on and blank until written, as the panel's U2 - confirm -> holds SDB high: the driver is on and blank until written, as the face board's - confirm
- R3: Confirm the wink left ladder resistor (DV24, L3-S1 11), on the plat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 -> the wink left ladder resistor (DV24, DP-CUR 7), on the boar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
- R4: Confirm the wink right ladder resistor (DV24, L3-S1 11), on the pla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 -> the wink right ladder resistor (DV24, DP-CUR 7), on the boa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
- SW1: footprint Button_Switch_THT:SW_PUSH_6mm -> cur-board:SW_PUSH_TL3342_Placeholder; Confirm 6 x 6 mm THT tactile under the faceplate's 17 x 15 cap (P19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 -> a TL3342-class 4.2 x 3.2 SMD tactile under the hatch cap (P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
- SW2: footprint Button_Switch_THT:SW_PUSH_6mm -> cur-board:SW_PUSH_TL3342_Placeholder; Confirm 6 x 6 mm THT tactile under the faceplate's 17 x 15 cap (P19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 -> a TL3342-class 4.2 x 3.2 SMD tactile under the fuel-door ca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
- SW3, SW4: Confirm P204: board-mount SPDT momentary under a lit 17 x 15 cap, C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 -> P204 (D-615): a subminiature SPDT momentary (Omron D2FS cla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
- SW5: Confirm P226: latching push button under a lit red-triangle 17 x 15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 -> P226 (D-615): a 5.8 mm self-locking push switch under the h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
- U1: Confirm the plate's LED driver (P199): fixed I2C address 0x54; VCC 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 -> the CUR's LED driver (P199): fixed I2C address 0x54; VCC 2.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
Connections:
- net AGND is gone; now on net WINK_COM: J1.8 (Pin_8)
- net JOY_PRESS is gone; now on net WINK_R_NC: J1.6 (Pin_6)
- net JOY_X is gone; now on net +5V_PNL: J1.4 (Pin_4)
- net JOY_Y is gone; now on net WINK_L_NC: J1.5 (Pin_5)
- net ROW1 is gone; now on net PNL_SDA: J1.1 (Pin_1)
- net +3V3: now also C3.1, C5.1, U2.24 (VDD), U3.5 (VOUT); no longer J1.7
- net +5V_PNL: now also C4.1, U3.1 (VIN), U3.3 (EN); no longer J1.12
- net GND: now also J1.3 (Pin_3), SW1.2, SW2.2, C3.2, C4.2, C5.2, ENC1.C, ENC1.S2, SW6.2 (COM), U2.12 (VSS), U2.2 (A1), U2.21 (A0), U2.3 (A2), U3.2 (GND); no longer J1.11
- net HAZ_LADDER: now also J1.9 (Pin_9)
- net KEY_FUEL: now also SW2.1, U2.9 (IO0_5); no longer SW2.2
- net KEY_HATCH: now also SW1.1, U2.8 (IO0_4); no longer SW1.2
- net PNL_SCL: now also J1.2 (Pin_2), U2.22 (SCL); no longer J1.10
- net PNL_SDA: now also U2.23 (SDA); no longer J1.9
- net WINK_REQ: now also J1.7 (Pin_7)
- removed net COL2: J1.2, SW1.1
- removed net COL3: J1.3, SW2.1
- new net KNOB_A: ENC1.A, U2.20 (IO1_7)
- new net KNOB_B: ENC1.B, U2.5 (IO0_1)
- new net KNOB_PUSH: ENC1.S1, U2.6 (IO0_2)
- new net MIR_DOWN: SW6.3 (DOWN), U2.15 (IO1_2)
- new net MIR_LEFT: SW6.6 (LEFT), U2.10 (IO0_6)
- new net MIR_PUSH: SW6.5 (PUSH), U2.7 (IO0_3)
- new net MIR_RIGHT: SW6.4 (RIGHT), U2.4 (IO0_0)
- new net MIR_UP: SW6.1 (UP), U2.19 (IO1_6)
- no-connect marks 12 -> 20
Other:
- note added: "0_4 hatch, 0_5 fuel door, 0_6 mirror left; IO1_2 mirror down,"
- note added: "1-4: the CU's I2C link (DP-DCU 44-47)."
- note added: "1_6 mirror up, 1_7 knob A. Its own 100 k pull-ups hold each high."
- note added: "5-9: the winks and the hazard, to the PMU box."
- note added: "AP2112K from +5V_PNL; under 1 mA drawn."
- note added: "Anodes on +5V_PNL, each in its cap or the well."
- note added: "D-597, D-615. Pad n = DP-CUR n."
- note added: "D-604, D-615. Each closes to GND; U2 reads it."
- note added: "Hazard: DP-CUR 9 -> 4.7k -> latching button -> commons; 47k across (D-368)."
- note added: "IO0_0 mirror right, 0_1 knob B, 0_2 knob push, 0_3 mirror push,"
- note added: "J1 - THE PIGTAIL TO DP-CUR"
- note added: "NC poles to DP-CUR 5 / 6, NO poles through 18k / 33k as WINK_REQ (DP-CUR 7),"
- note added: "Nine 20 AWG wires out through the rear grommet,"
- note added: "OUT1 wink L, OUT2 wink R, OUT3 hatch, OUT4 fuel,"
- note added: "OUT6 hazard, OUT13 mirror (lights.h). 7.6 mA."
- note added: "THE KEYS, THE MIRROR CONTROL, THE KNOB"
- note added: "THE SYMBOL LEDS"
- note added: "THE WINKS AND THE HAZARD (D-499, D-586, D-589)"
- note added: "The CU polls U2 over the bus: no INT wire."
- note added: "U1 - THE LIGHTS: IS31FL3218 at 0x54"
- note added: "U2 - THE I/O EXPANDER: PCA9555 at 0x20, on +3V3"
- note added: "U3 - 3.3 V FOR THE EXPANDER"
- note added: "the commons on DP-CUR 8 - the PMU box's star, NOT this board's GND."
- note added: "~150 mm to an inline DRC 24 - confirm."
- note removed: "Its red-triangle cap is LED6 on the driver's OUT6. The column's F-02 hazard contact is left unconnected (D-586)."
- note removed: "J1 - THE CABLE TO DP-DCU-E (P200)"
- note removed: "J4 - THE SCREEN KNOB'S LEAD (P219, D-580, D-581)"
- note removed: "L3-S1 6 (J2 pin 5) -> 4.7k -> the button -> the winks' commons (J2 pin 4, G20); 47k across the whole (D-368): the A8 ladder reads HAZARD while it is in."
- note removed: "NC poles to L3-S1 9 / 10 (J2 pins 1 / 2), NO poles through 18k / 33k joined as WINK_REQ to L3-S1 11 (J2 pin 3), the commons to dash ground (J2 pin 4, G20)."
- note removed: "OUT1 wink L face, OUT2 wink R face, OUT3 hatch, OUT4 fuel door, OUT6 hazard, OUT13 mirror stick - the DCU firmware's map (lights.h, F-018, Y62)"
- note removed: "OUT5, OUT7-OUT12, OUT14-OUT18 open. The bus pull-ups are on the carrier (R51 / R52, 4.7k to +3V3); none here."
- note removed: "ROW1 -> 1N4148W K..A -> key -> column"
- note removed: "STEMMA QT order: 1 GND, 2 +3V3, 3 PNL_SDA, 4 PNL_SCL. The knob's encoder board (seesaw 0x36) stands off the plate's front, its shaft through the faceplate."
- note removed: "THE HAZARD (P226, D-586, D-589): A LATCHING BUTTON ON THE WINK LEAD"
- note removed: "THE KEYS (matrix, D-492)"
- note removed: "THE LIGHTS: IS31FL3218 at 0x54, five symbols at 7.6 mA"
- note removed: "THE MIRROR STICK (P156, placeholder - no part chosen)"
- note removed: "THE WINK SWITCHES (P204, D-499) AND THEIR LEAD J2 TO THE DASH POST"
- note removed: "Two SPDT momentary pushbuttons under lit caps (the faces are LED1 / LED2 on the driver). Their lines are the harness's (DV24, D-189, D-482), unchanged:"
- note removed: "WINK_COM is NOT this board's GND: the winks return to the dash post as today, the plate's electronics on DP-DCU 43 and 46 (DV62). Symbol pins: 1 A = NC, 2 B = common, 3 C = NO."
- note removed: "hatch COL2 (DP-DCU-E 2), fuel door COL3 (DP-DCU-E 3)"
- note removed: "pin n = cavity n, on the net its panel_ribbon line names"
- note removed: "pots across +3V3 / AGND (D-380: its own return), wipers JOY_X / JOY_Y, the push JOY_PRESS to GND (panel_ribbon 19)"
- title: Left plate - the panel's second face, left of the steering wheel (D-492, D-499) -> CUR board - the Control Unit Remote (D-602, D-615)
- moved on the sheet: C1, C2, LED1, LED2, LED3, LED4, LED5, LED6, R1, R2, R3, R4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
